Commit message: Changed simulation parameters (dt,iter) and damping coefficient to improve stability

File: sr_description/hand/xacro/finger/biotac/biotac.urdf.xacro (robot description, xacro)
@@ -17,5 +17,6 @@
         <origin xyz="0 0 0.0125" rpy="0 0 0" />
         <mass value="0.012" />
-        <inertia  ixx="0.1" ixy="0.0"  ixz="0.0"  iyy="0.1"  iyz="0.0" izz="0.01" />
+      <inertia  ixx="0.00031" ixy="0.0"  ixz="0.0"  iyy="0.00031"  iyz="0.0"
+        izz="0.000053" />
       </inertial>
       <visual>
@@ -70,6 +71,6 @@
       <origin xyz="0 0 0.02" rpy="0 0 0" />
       <axis xyz="1 0 0" />
-      <limit lower="${20*M_PI/180}" upper="${20.1*M_PI/180}" effort="10" velocity="0.1" />
-      <dynamics damping="50.5"/>
+      <limit lower="${20*M_PI/180}" upper="${20.1*M_PI/180}" effort="2" velocity="0.1" />
+      <dynamics damping="0.1"/>
     </joint>
     <xacro:middle_transmission muscletrans="${muscle}" prefix="${prefix}" joint_prefix="${joint_prefix}" link_prefix="${link_prefix}"/>
@@ -122,5 +123,6 @@
        <mass value="0.001" />
        <origin xyz="0 0 0" rpy="0 0 0" />
-       <inertia  ixx="1" ixy="0"  ixz="0"  iyy="1"  iyz="0" izz="1" />
+        <inertia  ixx="0.00031" ixy="0.0"  ixz="0.0"  iyy="0.00031"  iyz="0.0"
+        izz="0.000053" />
       </inertial>
       <visual>

File: sr_description/hand/xacro/finger/distal/distal.urdf.xacro (robot description, xacro)
@@ -21,6 +21,6 @@
         <mass value="0.010" />
         <origin xyz="0 0 0.012" />
-        <inertia  ixx="0.0000031" ixy="0.0"  ixz="0.0"  iyy="0.0000031"  iyz="0.0"
-        izz="0.00000053" />
+        <inertia  ixx="0.00031" ixy="0.0"  ixz="0.0"  iyy="0.00031"  iyz="0.0"
+        izz="0.000053" />
       </inertial>
       <visual>
@@ -89,8 +89,8 @@
       <xacro:unless value="${bio}">
 				<!-- standard distal joint -->
-        <limit lower="0" upper="${M_PI/2}" effort="10"
+        <limit lower="0" upper="${M_PI/2}" effort="2"
           velocity="1.0" />
       </xacro:unless>
-      <dynamics damping="50.5"/>
+      <dynamics damping="0.1"/>
     </joint>
     <link name="${prefix}${link_prefix}tip">

File: sr_description/hand/xacro/finger/knuckle/knuckle.urdf.xacro (robot description, xacro)
@@ -19,5 +19,5 @@
         <!--<insert_block name="origin" /> -->
         <mass value="0.08" />
-        <inertia  ixx="0.000026" ixy="0.0"  ixz="0.0"  iyy="0.000026"  iyz="0.0"	izz="0.000032" />
+        <inertia  ixx="0.00026" ixy="0.0"  ixz="0.0"  iyy="0.00026"  iyz="0.0"	izz="0.00032" />
       </inertial>
       <visual>
@@ -42,6 +42,6 @@
       <insert_block name="axis"/>
       <limit lower="${-20/180*M_PI}" upper="${20/180*M_PI}"
-      effort="10" velocity="1.0"/>
-      <dynamics damping="50.5"/>
+      effort="2" velocity="1.0"/>
+      <dynamics damping="0.1"/>
     </joint>
     <!-- extensions -->

File: sr_description/hand/xacro/finger/lfmetacarpal/lfmetacarpal.urdf.xacro (robot description, xacro)
@@ -17,5 +17,5 @@
         <origin xyz="0 0 0.04" rpy="0 0 0" />
         <mass value="0.030" />
-	    <inertia  ixx="0.0000545" ixy="0.0"  ixz="0.0"  iyy="0.000056352"  iyz="0.0" izz="0.000004272" />
+	    <inertia  ixx="0.00545" ixy="0.0"  ixz="0.0"  iyy="0.0056352"  iyz="0.0" izz="0.0004272" />
       </inertial>
       <visual>
@@ -39,7 +39,7 @@
       <origin xyz="${reflect*-0.033} 0 0.02071" rpy="0 0 0" />
       <axis xyz="0.573576436 0 ${reflect*0.819152044}" />
-        <limit lower="0" upper="${45/180*M_PI}" effort="10"
+        <limit lower="0" upper="${45/180*M_PI}" effort="2"
       velocity="1.0" />
-      <dynamics damping="50.5"/>
+      <dynamics damping="0.1"/>
     </joint>
     <!-- extensions -->

File: sr_description/hand/xacro/finger/middle/middle.urdf.xacro (robot description, xacro)
@@ -18,6 +18,6 @@
         <origin xyz="0 0 0.0125" rpy="0 0 0" />
         <mass value="0.020" />
-        <inertia  ixx="0.0000067" ixy="0.0"  ixz="0.0"  iyy="0.0000067"  iyz="0.0"
-        izz="0.00000006" />
+        <inertia  ixx="0.00067" ixy="0.0"  ixz="0.0"  iyy="0.00067"  iyz="0.0"
+        izz="0.000006" />
       </inertial>
       <visual>
@@ -40,7 +40,7 @@
       <origin xyz="0 0 0.045" rpy="0 0 0" />
       <axis xyz="1 0 0" />
-      <limit lower="0" upper="${M_PI/2}" effort="10"
+      <limit lower="0" upper="${M_PI/2}" effort="2"
       velocity="1.0" />
-      <dynamics damping="50.5"/>
+      <dynamics damping="0.1"/>
     </joint>
     <!-- extensions -->

File: sr_description/hand/xacro/finger/proximal/proximal.urdf.xacro (robot description, xacro)
@@ -18,6 +18,6 @@
         <mass value="0.030" />
         <origin xyz="0 0 0.0225" />
-        <inertia  ixx="0.000037" ixy="0.0"  ixz="0.0"  iyy="0.000037"  iyz="0.0"
-        izz="0.00000018" />
+        <inertia  ixx="0.0037" ixy="0.0"  ixz="0.0"  iyy="0.0037"  iyz="0.0"
+        izz="0.000018" />
       </inertial>
       <visual>
@@ -40,7 +40,7 @@
       <origin xyz="0 0 0" rpy="0 0 0" />
       <axis xyz="1 0 0" />
-      <limit lower="0" upper="${M_PI/2}" effort="10"
+      <limit lower="0" upper="${M_PI/2}" effort="2"
       velocity="1.0"/>
-      <dynamics damping="50.5"/>
+      <dynamics damping="0.1"/>
     </joint>
     <!-- extensions -->

File: sr_description/hand/xacro/palm/palm.urdf.xacro (robot description, xacro)
@@ -17,5 +17,5 @@
         <origin xyz="0 0 0.035" rpy="0 0 0" />
         <mass value="0.3" />
-        <inertia  ixx="0.0003581" ixy="0.0"  ixz="0.0"  iyy="0.0005287"  iyz="0.0"	izz="0.0002545" />
+        <inertia  ixx="0.003581" ixy="0.0"  ixz="0.0"  iyy="0.005287"  iyz="0.0"	izz="0.002545" />
       </inertial>
       <visual>
@@ -41,5 +41,5 @@
       <limit lower="${-40/180*M_PI}" upper="${28/180*M_PI}"
       effort="5" velocity="1.0"/>
-      <dynamics damping="100.5"/>
+      <dynamics damping="0.1"/>
     </joint>
     <!-- extensions -->

File: sr_description/hand/xacro/wrist/wrist.urdf.xacro (robot description, xacro)
@@ -10,5 +10,5 @@
 		  <origin xyz="0 0 0" rpy="0 0 0" />
 		  <mass value="0.1" />
-		  <inertia  ixx="0.00120" ixy="0.0"  ixz="0.0"  iyy="0.00148"  iyz="0.0" izz="0.000438" />
+		  <inertia  ixx="0.0120" ixy="0.0"  ixz="0.0"  iyy="0.0148"  iyz="0.0" izz="0.00438" />
       </inertial>
       <visual>
@@ -36,6 +36,6 @@
       <insert_block name="origin" />
       <axis xyz="0 ${reflect} 0" />
-      <limit lower="${-30/180*M_PI}" upper="${10/180*M_PI}" effort="5" velocity="1.0"/>
-      <dynamics damping="100.5"/>
+      <limit lower="${-30/180*M_PI}" upper="${10/180*M_PI}" effort="3" velocity="1.0"/>
+      <dynamics damping="0.1"/>
     </joint>
     <!-- extensions -->

Commit message: Adapted dynamics damping parameter to be coherent with inertia retuned some joints to get nice movements

File: sr_description/hand/xacro/finger/biotac/biotac.urdf.xacro (robot description, xacro)
@@ -57,5 +57,5 @@
       <limit lower="0" upper="${M_PI/2}" effort="2.0"
       velocity="1.0" />
-      <dynamics damping="0.10"/>
+      <dynamics damping="0.001"/>
     </joint>
     <link name="${prefix}${link_prefix}_J1_dummy">
@@ -73,5 +73,5 @@
       <axis xyz="1 0 0" />
       <limit lower="${20*M_PI/180}" upper="${20.1*M_PI/180}" effort="1.0" velocity="1.0" />
-      <dynamics damping="0.1"/>
+      <dynamics damping="0.001"/>
     </joint>
     <xacro:middle_transmission muscletrans="${muscle}" prefix="${prefix}" joint_prefix="${joint_prefix}" link_prefix="${link_prefix}"/>

File: sr_description/hand/xacro/finger/distal/distal.urdf.xacro (robot description, xacro)
@@ -92,5 +92,5 @@
           velocity="1.0" />
       </xacro:unless>
-      <dynamics damping="0.1"/>
+      <dynamics damping="0.001"/>
     </joint>
     <link name="${prefix}${link_prefix}tip">

File: sr_description/hand/xacro/finger/knuckle/knuckle.urdf.xacro (robot description, xacro)
@@ -43,5 +43,5 @@
       <limit lower="${-20/180*M_PI}" upper="${20/180*M_PI}"
       effort="2" velocity="1.0"/>
-      <dynamics damping="0.1"/>
+      <dynamics damping="0.01"/>
     </joint>
     <!-- extensions -->

File: sr_description/hand/xacro/finger/lfmetacarpal/lfmetacarpal.urdf.xacro (robot description, xacro)
@@ -41,5 +41,5 @@
         <limit lower="0" upper="${45/180*M_PI}" effort="2"
       velocity="1.0" />
-      <dynamics damping="0.1"/>
+      <dynamics damping="0.001"/>
     </joint>
     <!-- extensions -->

File: sr_description/hand/xacro/finger/middle/middle.urdf.xacro (robot description, xacro)
@@ -54,5 +54,5 @@
       <limit lower="0" upper="${M_PI/2}" effort="2"
       velocity="1.0" />
-      <dynamics damping="0.1"/>
+      <dynamics damping="0.001"/>
     </joint>
     <!-- extensions -->

File: sr_description/hand/xacro/finger/proximal/proximal.urdf.xacro (robot description, xacro)
@@ -42,5 +42,5 @@
       <limit lower="0" upper="${M_PI/2}" effort="2"
       velocity="1.0"/>
-      <dynamics damping="0.1"/>
+      <dynamics damping="0.001"/>
     </joint>
     <!-- extensions -->

File: sr_description/hand/xacro/palm/palm.urdf.xacro (robot description, xacro)
@@ -82,5 +82,5 @@
       <limit lower="${-40/180*M_PI}" upper="${28/180*M_PI}"
       effort="30" velocity="1.0"/>
-      <dynamics damping="0.1"/>
+      <dynamics damping="0.01"/>
     </joint>
     <!-- extensions -->

File: sr_description/hand/xacro/thumb/thbase.urdf.xacro (robot description, xacro)
@@ -42,5 +42,5 @@
       <limit lower="${-60/180*M_PI}" upper="${60/180*M_PI}" effort="10"
       velocity="1.0" />
-      <dynamics damping="0.1"/>
+      <dynamics damping="0.001"/>
     </joint>
     <!-- extensions -->

File: sr_description/hand/xacro/thumb/thdistal.urdf.xacro (robot description, xacro)
@@ -31,5 +31,5 @@
 				<axis xyz="1 0 0" />
 				<limit lower="${20*M_PI/180}" upper="${20.1*M_PI/180}" effort="10" velocity="0.1" />
-				<dynamics damping="0.1"/>
+				<dynamics damping="0.001"/>
 			</joint>
 			<link name="${prefix}thbiotac">
@@ -165,5 +165,5 @@
 				<axis xyz="1 0 0" />
 				<limit lower="0" upper="${90.0*M_PI/180}" effort="10" velocity="1.0" />
-				<dynamics damping="0.1"/>
+				<dynamics damping="0.001"/>
 			</joint>
 			<link name="${prefix}thtip">

File: sr_description/hand/xacro/thumb/thhub.urdf.xacro (robot description, xacro)
@@ -53,5 +53,5 @@
         <limit lower="${-12/180*M_PI}" upper="${12/180*M_PI}" effort="10"
         velocity="1.0" />
-        <dynamics damping="0.1"/>
+        <dynamics damping="0.02"/>
       </joint>
     </xacro:unless>

File: sr_description/hand/xacro/thumb/thmiddle.urdf.xacro (robot description, xacro)
@@ -68,5 +68,5 @@
       <limit lower="${-40/180*M_PI}" upper="${40/180*M_PI}" effort="10"
       velocity="1.0" />
-      <dynamics damping="0.1"/>
+      <dynamics damping="0.001"/>
     </joint>
 		<!-- extensions -->

File: sr_description/hand/xacro/thumb/thproximal.urdf.xacro (robot description, xacro)
@@ -43,5 +43,5 @@
       <limit lower="0" upper="${70/180*M_PI}" effort="10"
       velocity="1.0" />
-      <dynamics damping="0.1"/>
+      <dynamics damping="0.005"/>
     </joint>
     <!-- extensions -->

File: sr_description/hand/xacro/wrist/wrist.urdf.xacro (robot description, xacro)
@@ -61,5 +61,5 @@
       <axis xyz="0 ${reflect} 0" />
       <limit lower="${-30/180*M_PI}" upper="${10/180*M_PI}" effort="30" velocity="1.0"/>
-      <dynamics damping="0.1"/>
+      <dynamics damping="0.01"/>
     </joint>
     <!-- extensions -->
