Commit message: Fixed thhub inertia (fixes strong THJ2 movement when THJ5 moves)

File: sr_description/hand/xacro/thumb/thhub.urdf.xacro (robot description, xacro)
@@ -18,6 +18,6 @@
 				<mass value="0.005" />
 				<origin xyz="0 0 0" rpy="0 0 0"/>
-				<inertia  ixx="0.0000001" ixy="0.0"  ixz="0.0"  iyy="0.0000001"  iyz="0.0"
-				izz="0.0000001" />
+				<inertia  ixx="0.000001" ixy="0.0"  ixz="0.0"  iyy="0.000001"  iyz="0.0"
+				izz="0.0000003" />
       </inertial>
       <visual>
