Commit message: Changed inertia values to real values, makes the hand collapse currently with gazebo 1.5 ODE

File: sr_description/hand/xacro/finger/distal/distal.urdf.xacro (robot description, xacro)
@@ -20,7 +20,7 @@
       <inertial>
         <mass value="0.010" />
-        <origin xyz="0 0 0.013" />
-        <inertia  ixx="0.1" ixy="0.0"  ixz="0.0"  iyy="0.1"  iyz="0.0"
-        izz="0.0" />
+        <origin xyz="0 0 0.012" />
+        <inertia  ixx="0.0000031" ixy="0.0"  ixz="0.0"  iyy="0.0000031"  iyz="0.0"
+        izz="0.00000053" />
       </inertial>
       <visual>

File: sr_description/hand/xacro/finger/knuckle/knuckle.urdf.xacro (robot description, xacro)
@@ -18,6 +18,6 @@
         <origin xyz="0 0 0" rpy="0 0 0" />
         <!--<insert_block name="origin" /> -->
-        <mass value="0.008" />
-        <inertia  ixx="0.0" ixy="0.0"  ixz="0.0"  iyy="0.1"  iyz="0.0"	izz="0.0" />
+        <mass value="0.08" />
+        <inertia  ixx="0.000026" ixy="0.0"  ixz="0.0"  iyy="0.000026"  iyz="0.0"	izz="0.000032" />
       </inertial>
       <visual>

File: sr_description/hand/xacro/finger/lfmetacarpal/lfmetacarpal.urdf.xacro (robot description, xacro)
@@ -16,6 +16,6 @@
       <inertial>
         <origin xyz="0 0 0.04" rpy="0 0 0" />
-        <mass value="0.075" />
-	    <inertia  ixx="0.1" ixy="0.0"  ixz="0.0"  iyy="0.1"  iyz="0.0" izz="0.1" />
+        <mass value="0.030" />
+	    <inertia  ixx="0.0000545" ixy="0.0"  ixz="0.0"  iyy="0.000056352"  iyz="0.0" izz="0.000004272" />
       </inertial>
       <visual>

File: sr_description/hand/xacro/finger/middle/middle.urdf.xacro (robot description, xacro)
@@ -17,7 +17,7 @@
       <inertial>
         <origin xyz="0 0 0.0125" rpy="0 0 0" />
-        <mass value="0.012" />
-        <inertia  ixx="0.1" ixy="0.0"  ixz="0.0"  iyy="0.1"  iyz="0.0"
-        izz="0.0" />
+        <mass value="0.020" />
+        <inertia  ixx="0.0000067" ixy="0.0"  ixz="0.0"  iyy="0.0000067"  iyz="0.0"
+        izz="0.00000006" />
       </inertial>
       <visual>

File: sr_description/hand/xacro/finger/proximal/proximal.urdf.xacro (robot description, xacro)
@@ -16,8 +16,8 @@
     <link name="${prefix}${link_prefix}proximal">
       <inertial>
-        <mass value="0.014" />
+        <mass value="0.030" />
         <origin xyz="0 0 0.0225" />
-        <inertia  ixx="0.1" ixy="0.0"  ixz="0.0"  iyy="0.1"  iyz="0.0"
-        izz="0.0" />
+        <inertia  ixx="0.000037" ixy="0.0"  ixz="0.0"  iyy="0.000037"  iyz="0.0"
+        izz="0.00000018" />
       </inertial>
       <visual>

File: sr_description/hand/xacro/forearm/forearm.urdf.xacro (robot description, xacro)
@@ -7,5 +7,5 @@
         <origin xyz="0 0 0.09" rpy="0 0 0"/>
         <mass value="3.0" />
-        <inertia  ixx="1.0" ixy="0.0"  ixz="0.0"  iyy="1.0"  iyz="0.0"  izz="1.0" />
+        <inertia  ixx="0.0108" ixy="0.0"  ixz="0.0"  iyy="0.0054"  iyz="0.0"  izz="0.0108" />
         </inertial>
         <visual>

File: sr_description/hand/xacro/palm/palm.urdf.xacro (robot description, xacro)
@@ -17,5 +17,5 @@
         <origin xyz="0 0 0.035" rpy="0 0 0" />
         <mass value="0.3" />
-        <inertia  ixx="0.5" ixy="0.0"  ixz="0.0"  iyy="0.5"  iyz="0.0"	izz="0.3" />
+        <inertia  ixx="0.0003581" ixy="0.0"  ixz="0.0"  iyy="0.0005287"  iyz="0.0"	izz="0.0002545" />
       </inertial>
       <visual>

File: sr_description/hand/xacro/wrist/wrist.urdf.xacro (robot description, xacro)
@@ -10,5 +10,5 @@
 		  <origin xyz="0 0 0" rpy="0 0 0" />
 		  <mass value="0.1" />
-		  <inertia  ixx="0.120" ixy="0.0"  ixz="0.0"  iyy="0.148"  iyz="0.0" izz="0.0438" />
+		  <inertia  ixx="0.00120" ixy="0.0"  ixz="0.0"  iyy="0.00148"  iyz="0.0" izz="0.000438" />
       </inertial>
       <visual>

Commit message: Made finger inertia homogeneous, otherwise the last joint vibrate due to small inertia Fixed correct thumb inertia and damping Retuned the hand in gazebo

File: sr_description/hand/xacro/finger/distal/distal.urdf.xacro (robot description, xacro)
@@ -21,6 +21,6 @@
         <mass value="0.010" />
         <origin xyz="0 0 0.012" />
-        <inertia  ixx="0.00031" ixy="0.0"  ixz="0.0"  iyy="0.00031"  iyz="0.0"
-        izz="0.000053" />
+        <inertia  ixx="0.001" ixy="0.0"  ixz="0.0"  iyy="0.001"  iyz="0.0"
+        izz="0.00025" />
       </inertial>
       <visual>

File: sr_description/hand/xacro/finger/knuckle/knuckle.urdf.xacro (robot description, xacro)
@@ -19,5 +19,5 @@
         <!--<insert_block name="origin" /> -->
         <mass value="0.08" />
-        <inertia  ixx="0.00026" ixy="0.0"  ixz="0.0"  iyy="0.00026"  iyz="0.0"	izz="0.00032" />
+        <inertia  ixx="0.0026" ixy="0.0"  ixz="0.0"  iyy="0.0026"  iyz="0.0"	izz="0.0032" />
       </inertial>
       <visual>

File: sr_description/hand/xacro/finger/middle/middle.urdf.xacro (robot description, xacro)
@@ -18,6 +18,6 @@
         <origin xyz="0 0 0.0125" rpy="0 0 0" />
         <mass value="0.020" />
-        <inertia  ixx="0.00067" ixy="0.0"  ixz="0.0"  iyy="0.00067"  iyz="0.0"
-        izz="0.000006" />
+        <inertia  ixx="0.002" ixy="0.0"  ixz="0.0"  iyy="0.002"  iyz="0.0"
+        izz="0.0002" />
       </inertial>
       <visual>

File: sr_description/hand/xacro/finger/proximal/proximal.urdf.xacro (robot description, xacro)
@@ -18,6 +18,6 @@
         <mass value="0.030" />
         <origin xyz="0 0 0.0225" />
-        <inertia  ixx="0.0037" ixy="0.0"  ixz="0.0"  iyy="0.0037"  iyz="0.0"
-        izz="0.000018" />
+        <inertia  ixx="0.003" ixy="0.0"  ixz="0.0"  iyy="0.003"  iyz="0.0"
+        izz="0.0003" />
       </inertial>
       <visual>

File: sr_description/hand/xacro/forearm/forearm.urdf.xacro (robot description, xacro)
@@ -7,5 +7,5 @@
         <origin xyz="0 0 0.09" rpy="0 0 0"/>
         <mass value="3.0" />
-        <inertia  ixx="0.0108" ixy="0.0"  ixz="0.0"  iyy="0.0054"  iyz="0.0"  izz="0.0108" />
+        <inertia  ixx="0.108" ixy="0.0"  ixz="0.0"  iyy="0.108"  iyz="0.0"  izz="0.054" />
         </inertial>
         <visual>
@@ -33,5 +33,5 @@
             <origin xyz="0 0 0.09" rpy="0 0 0" />
             <geometry name="${prefix}forearm_collision">
-              <cylinder radius="0.07" length="0.180"/>
+              <box size="0.140 0.140 0.180" />
             </geometry>
           </xacro:unless>

File: sr_description/hand/xacro/palm/palm.urdf.xacro (robot description, xacro)
@@ -40,5 +40,5 @@
       <axis xyz="1 0 0" />
       <limit lower="${-40/180*M_PI}" upper="${28/180*M_PI}"
-      effort="5" velocity="1.0"/>
+      effort="30" velocity="1.0"/>
       <dynamics damping="0.1"/>
     </joint>

File: sr_description/hand/xacro/thumb/thbase.urdf.xacro (robot description, xacro)
@@ -17,6 +17,6 @@
 				<mass value="0.010" />
 				<origin xyz="0 0 0" rpy="0 0 0"/>
-				<inertia  ixx="0.0" ixy="0.0"  ixz="0.0"  iyy="0.0"  iyz="0.0" izz="0.1" />
-      </inertial>
+				<inertia  ixx="0.0003" ixy="0.0"  ixz="0.0"  iyy="0.0003"  iyz="0.0" izz="0.0003" />
+			</inertial>
       <visual>
 				<origin xyz="0 0 0" rpy="0 0 0" />
@@ -42,5 +42,5 @@
       <limit lower="${-60/180*M_PI}" upper="${60/180*M_PI}" effort="10"
       velocity="1.0" />
-      <dynamics damping="50.5"/>
+      <dynamics damping="0.1"/>
     </joint>
     <!-- extensions -->

File: sr_description/hand/xacro/thumb/thdistal.urdf.xacro (robot description, xacro)
@@ -21,6 +21,7 @@
 					<origin xyz="0 0 0" rpy="0 0 0" />
 					<mass value="0.01" />
-					<inertia  ixx="0.1" ixy="0.0"  ixz="0.0"  iyy="0.1"  iyz="0.0" izz="0.01" />
-				</inertial>
+					 <inertia  ixx="0.0007" ixy="0.0"  ixz="0.0"  iyy="0.0007"  iyz="0.0"
+        izz="0.00010" />
+        </inertial>
 			</link>
 			<joint name="${prefix}THJ1" type="revolute">
@@ -30,5 +31,5 @@
 				<axis xyz="1 0 0" />
 				<limit lower="${20*M_PI/180}" upper="${20.1*M_PI/180}" effort="10" velocity="0.1" />
-				<dynamics damping="50.5"/>
+				<dynamics damping="0.1"/>
 			</joint>
 			<link name="${prefix}thbiotac">
@@ -36,5 +37,6 @@
 					<origin xyz="0 0 0" rpy="0 0 0" />
 					<mass value="0.2" />
-					<inertia  ixx="1" ixy="0.0"  ixz="0.0"  iyy="1"  iyz="0.0" izz="1" />
+					 <inertia  ixx="0.0007" ixy="0.0"  ixz="0.0"  iyy="0.0007"  iyz="0.0"
+        izz="0.00010" />
 				</inertial>
 				<visual>
@@ -80,5 +82,5 @@
 				 <mass value="0.001" />
 				 <origin xyz="0 0 0" rpy="0 0 0" />
-				 <inertia  ixx="1" ixy="0"  ixz="0"  iyy="1"  iyz="0" izz="1" />
+				 <inertia  ixx="0" ixy="0"  ixz="0"  iyy="0"  iyz="0" izz="0" />
 				</inertial>
 				<visual>
@@ -108,6 +110,6 @@
 					<mass value="0.016" />
 					<origin xyz="0 0 0.01375" rpy="0 0 0"/>
-					<inertia  ixx="0.1" ixy="0.0"  ixz="0.0"  iyy="0.1"  iyz="0.0"
-							izz="0.1" />
+					 <inertia  ixx="0.0007" ixy="0.0"  ixz="0.0"  iyy="0.0007"  iyz="0.0"
+        izz="0.00010" />
 				</inertial>
 				<visual>
@@ -160,5 +162,5 @@
 				<axis xyz="1 0 0" />
 				<limit lower="0" upper="${90.0*M_PI/180}" effort="10" velocity="1.0" />
-				<dynamics damping="50.5"/>
+				<dynamics damping="0.1"/>
 			</joint>
 			<link name="${prefix}thtip">

File: sr_description/hand/xacro/thumb/thhub.urdf.xacro (robot description, xacro)
@@ -15,8 +15,8 @@
     <link name="${prefix}thhub">
       <inertial>
-				<mass value="0.002" />
+				<mass value="0.01" />
 				<origin xyz="0 0 0" rpy="0 0 0"/>
-				<inertia  ixx="0.1" ixy="0.0"  ixz="0.0"  iyy="0.1"  iyz="0.0"
-				izz="0.1" />
+				<inertia  ixx="0.0003" ixy="0.0"  ixz="0.0"  iyy="0.0003"  iyz="0.0"
+				izz="0.0003" />
       </inertial>
       <visual>
@@ -43,5 +43,5 @@
       <limit lower="${-12/180*M_PI}" upper="${12/180*M_PI}" effort="10"
       velocity="1.0" />
-      <dynamics damping="50.5"/>
+      <dynamics damping="0.1"/>
     </joint>
 		<!-- extensions -->

File: sr_description/hand/xacro/thumb/thmiddle.urdf.xacro (robot description, xacro)
@@ -15,8 +15,8 @@
     <link name="${prefix}thmiddle">
       <inertial>
-				<mass value="0.016" />
+				<mass value="0.027" />
 				<origin xyz="0 0 0.016" rpy="0 0 0"/>
-				<inertia  ixx="0.1" ixy="0.0"  ixz="0.0"  iyy="0.1"  iyz="0.0"
-				izz="0.1" />
+				<inertia  ixx="0.0026" ixy="0.0"  ixz="0.0"  iyy="0.0026"  iyz="0.0"
+				izz="0.000169" />
       </inertial>
       <visual>
@@ -61,5 +61,5 @@
       <limit lower="${-40/180*M_PI}" upper="${40/180*M_PI}" effort="10"
       velocity="1.0" />
-      <dynamics damping="50.5"/>
+      <dynamics damping="0.1"/>
     </joint>
 		<!-- extensions -->

File: sr_description/hand/xacro/thumb/thproximal.urdf.xacro (robot description, xacro)
@@ -15,8 +15,9 @@
     <link name="${prefix}thproximal">
       <inertial>
-				<mass value="0.016" />
+				<mass value="0.040" />
 				<origin xyz="0 0 0.019" rpy="0 0 0"/>
-				<inertia  ixx="0.1" ixy="0.0"  ixz="0.0"  iyy="0.1"  iyz="0.0"	izz="0.1" />
-      </inertial>
+					<inertia  ixx="0.00496" ixy="0.0"  ixz="0.0"  iyy="0.00496"  iyz="0.0"
+				izz="0.000312" />
+			</inertial>
       <visual>
 				<origin xyz="0 0 0" rpy="0 0 0" />
@@ -42,5 +43,5 @@
       <limit lower="0" upper="${70/180*M_PI}" effort="10"
       velocity="1.0" />
-      <dynamics damping="50.5"/>
+      <dynamics damping="0.1"/>
     </joint>
     <!-- extensions -->

File: sr_description/hand/xacro/wrist/wrist.urdf.xacro (robot description, xacro)
@@ -36,5 +36,5 @@
       <insert_block name="origin" />
       <axis xyz="0 ${reflect} 0" />
-      <limit lower="${-30/180*M_PI}" upper="${10/180*M_PI}" effort="3" velocity="1.0"/>
+      <limit lower="${-30/180*M_PI}" upper="${10/180*M_PI}" effort="30" velocity="1.0"/>
       <dynamics damping="0.1"/>
     </joint>

Commit message: Tested real inertia in gazebo indigo

File: sr_description/hand/xacro/finger/distal/distal.urdf.xacro (robot description, xacro)
@@ -21,6 +21,6 @@
         <mass value="0.010" />
         <origin xyz="0 0 0.012" />
-        <inertia  ixx="0.001" ixy="0.0"  ixz="0.0"  iyy="0.001"  iyz="0.0"
-        izz="0.00025" />
+        <inertia  ixx="0.0000031" ixy="0.0"  ixz="0.0"  iyy="0.0000031"  iyz="0.0"
+        izz="0.00000053" />
       </inertial>
       <visual>

File: sr_description/hand/xacro/finger/knuckle/knuckle.urdf.xacro (robot description, xacro)
@@ -19,5 +19,5 @@
         <!--<insert_block name="origin" /> -->
         <mass value="0.08" />
-        <inertia  ixx="0.0026" ixy="0.0"  ixz="0.0"  iyy="0.0026"  iyz="0.0"	izz="0.0032" />
+        <inertia  ixx="0.000026" ixy="0.0"  ixz="0.0"  iyy="0.000026"  iyz="0.0"	izz="0.000032" />
       </inertial>
       <visual>

File: sr_description/hand/xacro/finger/lfmetacarpal/lfmetacarpal.urdf.xacro (robot description, xacro)
@@ -17,5 +17,5 @@
         <origin xyz="0 0 0.04" rpy="0 0 0" />
         <mass value="0.030" />
-	    <inertia  ixx="0.00545" ixy="0.0"  ixz="0.0"  iyy="0.0056352"  iyz="0.0" izz="0.0004272" />
+	    <inertia  ixx="0.0000545" ixy="0.0"  ixz="0.0"  iyy="0.000056352"  iyz="0.0" izz="0.000004272" />
       </inertial>
       <visual>

File: sr_description/hand/xacro/finger/middle/middle.urdf.xacro (robot description, xacro)
@@ -18,6 +18,6 @@
         <origin xyz="0 0 0.0125" rpy="0 0 0" />
         <mass value="0.020" />
-        <inertia  ixx="0.002" ixy="0.0"  ixz="0.0"  iyy="0.002"  iyz="0.0"
-        izz="0.0002" />
+        <inertia  ixx="0.0000067" ixy="0.0"  ixz="0.0"  iyy="0.0000067"  iyz="0.0"
+        izz="0.00000006" />
       </inertial>
       <visual>

File: sr_description/hand/xacro/finger/proximal/proximal.urdf.xacro (robot description, xacro)
@@ -18,6 +18,6 @@
         <mass value="0.030" />
         <origin xyz="0 0 0.0225" />
-        <inertia  ixx="0.003" ixy="0.0"  ixz="0.0"  iyy="0.003"  iyz="0.0"
-        izz="0.0003" />
+        <inertia  ixx="0.000037" ixy="0.0"  ixz="0.0"  iyy="0.000037"  iyz="0.0"
+        izz="0.00000018" />
       </inertial>
       <visual>

File: sr_description/hand/xacro/forearm/forearm.urdf.xacro (robot description, xacro)
@@ -7,5 +7,5 @@
         <origin xyz="0 0 0.09" rpy="0 0 0"/>
         <mass value="3.0" />
-        <inertia  ixx="0.108" ixy="0.0"  ixz="0.0"  iyy="0.108"  iyz="0.0"  izz="0.054" />
+        <inertia  ixx="0.0138" ixy="0.0"  ixz="0.0"  iyy="0.0138"  iyz="0.0"  izz="0.00744" />
         </inertial>
         <visual>

File: sr_description/hand/xacro/palm/palm.urdf.xacro (robot description, xacro)
@@ -17,5 +17,5 @@
         <origin xyz="0 0 0.035" rpy="0 0 0" />
         <mass value="0.3" />
-        <inertia  ixx="0.003581" ixy="0.0"  ixz="0.0"  iyy="0.005287"  iyz="0.0"	izz="0.002545" />
+        <inertia  ixx="0.0003581" ixy="0.0"  ixz="0.0"  iyy="0.0005287"  iyz="0.0"	izz="0.0002545" />
       </inertial>
       <visual>

File: sr_description/hand/xacro/wrist/wrist.urdf.xacro (robot description, xacro)
@@ -10,5 +10,5 @@
 		  <origin xyz="0 0 0" rpy="0 0 0" />
 		  <mass value="0.1" />
-		  <inertia  ixx="0.0120" ixy="0.0"  ixz="0.0"  iyy="0.0148"  iyz="0.0" izz="0.00438" />
+		  <inertia  ixx="0.000024" ixy="0.0"  ixz="0.0"  iyy="0.000104"  iyz="0.0" izz="0.0000867" />
       </inertial>
       <visual>
