Commit message: Set inertia to suggested ones by HSU, set back the damping, effort and velocity to old values (although completely unrealistic)

File: sr_description/hand/xacro/finger/distal/distal.urdf.xacro (robot description, xacro)
@@ -21,6 +21,6 @@
         <mass value="0.010" />
         <origin xyz="0 0 0.012" />
-        <inertia  ixx="0.001" ixy="0.0"  ixz="0.0"  iyy="0.001"  iyz="0.0"
-        izz="0.00025" />
+        <inertia  ixx="0.0000001" ixy="0.0"  ixz="0.0"  iyy="0.0000001"  iyz="0.0"
+        izz="0.0000001" />
       </inertial>
       <visual>
@@ -84,18 +84,18 @@
       <xacro:if value="${bio}">
 				<!-- biotac fixed distal joint -->
-        <limit lower="${20/180*M_PI}" upper="${20/180*M_PI}" effort="10"
-          velocity="1.0" />
+        <limit lower="${20/180*M_PI}" upper="${20/180*M_PI}" effort="1000"
+          velocity="10.0" />
       </xacro:if>
       <xacro:unless value="${bio}">
 				<!-- standard distal joint -->
-        <limit lower="0" upper="${M_PI/2}" effort="2"
-          velocity="1.0" />
+        <limit lower="0" upper="${M_PI/2}" effort="1000"
+          velocity="10.0" />
       </xacro:unless>
-      <dynamics damping="0.1"/>
+      <dynamics damping="1.0"/>
     </joint>
     <link name="${prefix}${link_prefix}tip">
 			<inertial>
 				<mass value="0.001" />
-				<inertia  ixx="0.0" ixy="0.0"  ixz="0.0"  iyy="0.0"  iyz="0.0" izz="0.0" />
+				<inertia  ixx="0.0000001" ixy="0.0"  ixz="0.0"  iyy="0.0000001"  iyz="0.0" izz="0.0000001" />
   		</inertial>
     </link>

File: sr_description/hand/xacro/finger/knuckle/knuckle.urdf.xacro (robot description, xacro)
@@ -18,6 +18,6 @@
         <origin xyz="0 0 0" rpy="0 0 0" />
         <!--<insert_block name="origin" /> -->
-        <mass value="0.08" />
-        <inertia  ixx="0.0026" ixy="0.0"  ixz="0.0"  iyy="0.0026"  iyz="0.0"	izz="0.0032" />
+        <mass value="0.008" />
+        <inertia  ixx="0.0000002" ixy="0.0"  ixz="0.0"  iyy="0.0000002"  iyz="0.0"	izz="0.0000002" />
       </inertial>
       <visual>
@@ -42,6 +42,6 @@
       <insert_block name="axis"/>
       <limit lower="${-20/180*M_PI}" upper="${20/180*M_PI}"
-      effort="2" velocity="1.0"/>
-      <dynamics damping="0.1"/>
+      effort="1000" velocity="10.0"/>
+      <dynamics damping="1.0"/>
     </joint>
     <!-- extensions -->

File: sr_description/hand/xacro/finger/lfmetacarpal/lfmetacarpal.urdf.xacro (robot description, xacro)
@@ -17,5 +17,5 @@
         <origin xyz="0 0 0.04" rpy="0 0 0" />
         <mass value="0.030" />
-	    <inertia  ixx="0.00545" ixy="0.0"  ixz="0.0"  iyy="0.0056352"  iyz="0.0" izz="0.0004272" />
+	    <inertia  ixx="5e-6" ixy="0.0"  ixz="0.0"  iyy="5e-6"  iyz="0.0" izz="3e-6" />
       </inertial>
       <visual>
@@ -39,7 +39,7 @@
       <origin xyz="${reflect*-0.033} 0 0.02071" rpy="0 0 0" />
       <axis xyz="0.573576436 0 ${reflect*0.819152044}" />
-        <limit lower="0" upper="${45/180*M_PI}" effort="2"
-      velocity="1.0" />
-      <dynamics damping="0.1"/>
+        <limit lower="0" upper="${45/180*M_PI}" effort="1000"
+      velocity="10.0" />
+      <dynamics damping="1.0"/>
     </joint>
     <!-- extensions -->

File: sr_description/hand/xacro/finger/middle/middle.urdf.xacro (robot description, xacro)
@@ -18,6 +18,6 @@
         <origin xyz="0 0 0.0125" rpy="0 0 0" />
         <mass value="0.020" />
-        <inertia  ixx="0.002" ixy="0.0"  ixz="0.0"  iyy="0.002"  iyz="0.0"
-        izz="0.0002" />
+        <inertia  ixx="0.0000008" ixy="0.0"  ixz="0.0"  iyy="0.0000008"  iyz="0.0"
+        izz="0.0000003" />
       </inertial>
       <visual>
@@ -52,7 +52,7 @@
       <origin xyz="0 0 0.045" rpy="0 0 0" />
       <axis xyz="1 0 0" />
-      <limit lower="0" upper="${M_PI/2}" effort="2"
-      velocity="1.0" />
-      <dynamics damping="0.1"/>
+      <limit lower="0" upper="${M_PI/2}" effort="1000"
+      velocity="10.0" />
+      <dynamics damping="1.0"/>
     </joint>
     <!-- extensions -->

File: sr_description/hand/xacro/finger/proximal/proximal.urdf.xacro (robot description, xacro)
@@ -18,6 +18,6 @@
         <mass value="0.030" />
         <origin xyz="0 0 0.0225" />
-        <inertia  ixx="0.003" ixy="0.0"  ixz="0.0"  iyy="0.003"  iyz="0.0"
-        izz="0.0003" />
+        <inertia  ixx="0.0000010" ixy="0.0"  ixz="0.0"  iyy="0.0000010"  iyz="0.0"
+        izz="0.0000005" />
       </inertial>
       <visual>
@@ -40,7 +40,7 @@
       <origin xyz="0 0 0" rpy="0 0 0" />
       <axis xyz="1 0 0" />
-      <limit lower="0" upper="${M_PI/2}" effort="2"
-      velocity="1.0"/>
-      <dynamics damping="0.1"/>
+      <limit lower="0" upper="${M_PI/2}" effort="1000"
+      velocity="10.0"/>
+      <dynamics damping="1.0"/>
     </joint>
     <!-- extensions -->

File: sr_description/hand/xacro/forearm/forearm.urdf.xacro (robot description, xacro)
@@ -7,5 +7,5 @@
         <origin xyz="0 0 0.09" rpy="0 0 0"/>
         <mass value="3.0" />
-        <inertia  ixx="0.108" ixy="0.0"  ixz="0.0"  iyy="0.108"  iyz="0.0"  izz="0.054" />
+        <inertia  ixx="0.001" ixy="0.0"  ixz="0.0"  iyy="0.001"  iyz="0.0"  izz="0.001" />
         </inertial>
         <visual>

File: sr_description/hand/xacro/palm/palm.urdf.xacro (robot description, xacro)
@@ -17,5 +17,5 @@
         <origin xyz="0 0 0.035" rpy="0 0 0" />
         <mass value="0.3" />
-        <inertia  ixx="0.003581" ixy="0.0"  ixz="0.0"  iyy="0.005287"  iyz="0.0"	izz="0.002545" />
+        <inertia  ixx="0.00013581" ixy="0.0"  ixz="0.0"  iyy="0.000185"  iyz="0.0"	izz="0.0000725" />
       </inertial>
       <visual>
@@ -81,6 +81,6 @@
       <axis xyz="1 0 0" />
       <limit lower="${-40/180*M_PI}" upper="${28/180*M_PI}"
-      effort="30" velocity="1.0"/>
-      <dynamics damping="0.1"/>
+      effort="1000" velocity="10.0"/>
+      <dynamics damping="1.0"/>
     </joint>
     <!-- extensions -->

File: sr_description/hand/xacro/thumb/thbase.urdf.xacro (robot description, xacro)
@@ -17,5 +17,5 @@
 				<mass value="0.010" />
 				<origin xyz="0 0 0" rpy="0 0 0"/>
-				<inertia  ixx="0.0003" ixy="0.0"  ixz="0.0"  iyy="0.0003"  iyz="0.0" izz="0.0003" />
+				<inertia  ixx="1e-6" ixy="0.0"  ixz="0.0"  iyy="1e-6"  iyz="0.0" izz="1e-6" />
 			</inertial>
       <visual>
@@ -40,7 +40,7 @@
       <origin xyz="${reflect*0.034} -0.0085 0.029" rpy="0 ${M_PI/4} ${M_PI/2-reflect*M_PI/2}" />
       <axis xyz="0 0 ${reflect*-1}" />
-      <limit lower="${-60/180*M_PI}" upper="${60/180*M_PI}" effort="10"
-      velocity="1.0" />
-      <dynamics damping="0.1"/>
+      <limit lower="${-60/180*M_PI}" upper="${60/180*M_PI}" effort="1000"
+      velocity="10.0" />
+      <dynamics damping="1.0"/>
     </joint>
     <!-- extensions -->

File: sr_description/hand/xacro/thumb/thdistal.urdf.xacro (robot description, xacro)
@@ -113,6 +113,6 @@
 					<mass value="0.016" />
 					<origin xyz="0 0 0.01375" rpy="0 0 0"/>
-					 <inertia  ixx="0.0007" ixy="0.0"  ixz="0.0"  iyy="0.0007"  iyz="0.0"
-        izz="0.00010" />
+					 <inertia  ixx="9e-7" ixy="0.0"  ixz="0.0"  iyy="9e-7"  iyz="0.0"
+        izz="9e-7" />
 				</inertial>
 				<visual>
@@ -164,11 +164,11 @@
 				<origin xyz="0 0 0.032" rpy="0 0 ${-M_PI/2}" />
 				<axis xyz="1 0 0" />
-				<limit lower="0" upper="${90.0*M_PI/180}" effort="10" velocity="1.0" />
-				<dynamics damping="0.1"/>
+				<limit lower="0" upper="${90.0*M_PI/180}" effort="1000" velocity="10.0" />
+				<dynamics damping="1.0"/>
 			</joint>
 			<link name="${prefix}thtip">
 				<inertial>
 					<mass value="0.001" />
-					<inertia  ixx="0.0" ixy="0.0"  ixz="0.0"  iyy="0.0"  iyz="0.0" izz="0.0" />
+					<inertia  ixx="1e-7" ixy="0.0"  ixz="0.0"  iyy="1e-7"  iyz="0.0" izz="1e-7" />
 				</inertial>
 			</link>

File: sr_description/hand/xacro/thumb/thhub.urdf.xacro (robot description, xacro)
@@ -16,8 +16,8 @@
     <link name="${prefix}thhub">
       <inertial>
-				<mass value="0.01" />
+				<mass value="0.002" />
 				<origin xyz="0 0 0" rpy="0 0 0"/>
-				<inertia  ixx="0.0003" ixy="0.0"  ixz="0.0"  iyy="0.0003"  iyz="0.0"
-				izz="0.0003" />
+				<inertia  ixx="1e-7" ixy="0.0"  ixz="0.0"  iyy="1e-7"  iyz="0.0"
+				izz="1e-7" />
       </inertial>
       <visual>
@@ -51,7 +51,7 @@
         <origin xyz="0 0 0.038" rpy="0 0 0" />
         <axis xyz="1 0 0" />
-        <limit lower="${-12/180*M_PI}" upper="${12/180*M_PI}" effort="10"
-        velocity="1.0" />
-        <dynamics damping="0.1"/>
+        <limit lower="${-12/180*M_PI}" upper="${12/180*M_PI}" effort="1000"
+        velocity="10.0" />
+        <dynamics damping="1.0"/>
       </joint>
     </xacro:unless>

File: sr_description/hand/xacro/thumb/thmiddle.urdf.xacro (robot description, xacro)
@@ -17,5 +17,5 @@
         <mass value="0.027" />
         <origin xyz="0 0 0.016" rpy="0 0 0"/>
-          <inertia  ixx="0.0026" ixy="0.0"  ixz="0.0"  iyy="0.0026"  iyz="0.0" izz="0.000169" />
+          <inertia  ixx="1e-6" ixy="0.0"  ixz="0.0"  iyy="1e-6"  iyz="0.0" izz="1e-6" />
       </inertial>
       <visual>
@@ -66,7 +66,7 @@
 				</xacro:unless>
       <axis xyz="0 -1 0" />
-      <limit lower="${-40/180*M_PI}" upper="${40/180*M_PI}" effort="10"
-      velocity="1.0" />
-      <dynamics damping="0.1"/>
+      <limit lower="${-40/180*M_PI}" upper="${40/180*M_PI}" effort="1000"
+      velocity="10.0" />
+      <dynamics damping="1.0"/>
     </joint>
 		<!-- extensions -->

File: sr_description/hand/xacro/thumb/thproximal.urdf.xacro (robot description, xacro)
@@ -15,8 +15,8 @@
     <link name="${prefix}thproximal">
       <inertial>
-				<mass value="0.040" />
+				<mass value="0.016" />
 				<origin xyz="0 0 0.019" rpy="0 0 0"/>
-					<inertia  ixx="0.00496" ixy="0.0"  ixz="0.0"  iyy="0.00496"  iyz="0.0"
-				izz="0.000312" />
+					<inertia  ixx="1e-6" ixy="0.0"  ixz="0.0"  iyy="1e-6"  iyz="0.0"
+				izz="1e-6" />
 			</inertial>
       <visual>
@@ -41,7 +41,6 @@
       <origin xyz="0 0 0" rpy="0 0 0" />
       <axis xyz="${reflect} 0 0" />
-      <limit lower="0" upper="${70/180*M_PI}" effort="10"
-      velocity="1.0" />
-      <dynamics damping="0.1"/>
+      <limit lower="0" upper="${70/180*M_PI}" effort="1000"      velocity="10.0" />
+      <dynamics damping="1.0"/>
     </joint>
     <!-- extensions -->

File: sr_description/hand/xacro/wrist/wrist.urdf.xacro (robot description, xacro)
@@ -10,5 +10,5 @@
 		  <origin xyz="0 0 0" rpy="0 0 0" />
 		  <mass value="0.1" />
-		  <inertia  ixx="0.0120" ixy="0.0"  ixz="0.0"  iyy="0.0148"  iyz="0.0" izz="0.00438" />
+		  <inertia  ixx="0.000120" ixy="0.0"  ixz="0.0"  iyy="0.000148"  iyz="0.0" izz="0.0000438" />
       </inertial>
       <visual>
@@ -60,6 +60,6 @@
       <insert_block name="origin" />
       <axis xyz="0 ${reflect} 0" />
-      <limit lower="${-30/180*M_PI}" upper="${10/180*M_PI}" effort="30" velocity="1.0"/>
-      <dynamics damping="0.1"/>
+      <limit lower="${-30/180*M_PI}" upper="${10/180*M_PI}" effort="1000" velocity="10.0"/>
+      <dynamics damping="1.0"/>
     </joint>
     <!-- extensions -->

Commit message: Changed ubi fingertip meshes and taxels, adapted distal phalanx to use them

File: sr_description/hand/xacro/finger/distal/distal.urdf.xacro (robot description, xacro)
@@ -29,5 +29,5 @@
           <xacro:if value="${ubi}">
 			<!-- Ubi distal -->
-            <mesh filename="package://sr_description/hand/model/F1.dae" scale="0.001 0.001 0.001" />
+            <mesh filename="package://sr_description/hand/model/ubi_tactiles/ubi_tip_visual.dae" scale="0.001 0.001 0.001" />
           </xacro:if>
           <xacro:unless value="${ubi}">
@@ -55,5 +55,5 @@
           <xacro:if value="${ubi}">
 						<!-- Ubi distal -->
-            <mesh filename="package://sr_description/hand/model/F1.dae" scale="0.001 0.001 0.001" />
+            <mesh filename="package://sr_description/hand/model/ubi_tactiles/ubi_tip_collision.dae" scale="0.001 0.001 0.001" />
           </xacro:if>
           <xacro:unless value="${ubi}">
