Commit message: Inertia now exact values, with inertia tensor at COM (gazebo and ode support the small values now) Removed explicit viscous damping from sr_gazebo_plugin, enabled springDamper in each joint (implicit viscous damping) changed simulation parameters for stability and retuned the controllers, explicitely define friction_deadband for simulated controllers (default is for real hand and is too high)

File: sr_description/arm/xacro/base/shadowarm_base.urdf.xacro (robot description, xacro)
@@ -6,5 +6,5 @@
       <origin xyz="0 0 0" rpy="0 0 0"/>
       <mass value="0.4" />
-      <inertia  ixx="0.1" ixy="0.0"  ixz="0.0"  iyy="0.1"  iyz="0.0"  izz="0.1" />
+      <inertia  ixx="0.00071" ixy="0.0"  ixz="0.0"  iyy="0.00071"  iyz="0.0"  izz="0.0014" />
     </inertial>
     <visual>

File: sr_description/arm/xacro/hand_support/shadowarm_handsupport_motor.urdf.xacro (robot description, xacro)
@@ -6,5 +6,5 @@
 	<origin xyz="0 0 0" rpy="0 0 0" />
 	<mass value="0.75" />
-	<inertia  ixx="0.01" ixy="0.0"  ixz="0.0"  iyy="0.01"  iyz="0.0"  izz="0.016" />
+	<inertia  ixx="0.00086" ixy="0.0"  ixz="0.0"  iyy="0.00086"  iyz="0.0"  izz="0.0017" />
       </inertial>
       <visual>
@@ -35,4 +35,8 @@
       <dynamics damping="5.5"/>
     </joint>
+    <gazebo reference="ElbowJRotate">
+      <provideFeedback>1</provideFeedback>
+      <implicitSpringDamper>1</implicitSpringDamper>
+    </gazebo>
     <xacro:shadowarm_handsupport_motor_transmission />
   </xacro:macro>

File: sr_description/arm/xacro/hand_support/shadowarm_handsupport_muscle.urdf.xacro (robot description, xacro)
@@ -6,5 +6,5 @@
 	<origin xyz="0 0 0" rpy="0 0 0" />
 	<mass value="0.75" />
-	<inertia  ixx="0.01" ixy="0.0"  ixz="0.0"  iyy="0.01"  iyz="0.0"  izz="0.016" />
+	<inertia  ixx="0.00092" ixy="0.0"  ixz="0.0"  iyy="0.00092"  iyz="0.0"  izz="0.0018" />
       </inertial>
       <visual>
@@ -35,4 +35,8 @@
       <dynamics damping="5.5"/>
     </joint>
+    <gazebo reference="ElbowJRotate">
+      <provideFeedback>1</provideFeedback>
+      <implicitSpringDamper>1</implicitSpringDamper>
+    </gazebo>
     <xacro:shadowarm_handsupport_muscle_transmission />
   </xacro:macro>

File: sr_description/arm/xacro/lower_arm/shadowarm_lowerarm.urdf.xacro (robot description, xacro)
@@ -6,5 +6,5 @@
 	  <origin xyz="0.08 0 0.0625" rpy="0 0 0" />
 	  <mass value="1.7" />
-	  <inertia  ixx="0.01" ixy="0.0"  ixz="0.0"  iyy="0.01"  iyz="0.0"  izz="0.01" />
+	  <inertia  ixx="0.0016" ixy="0.0"  ixz="0.0"  iyy="0.0016"  iyz="0.0"  izz="0.0018" />
 	</inertial>
 	<visual>
@@ -35,4 +35,8 @@
       <dynamics damping="5.5"/>
     </joint>
+    <gazebo reference="ElbowJSwing">
+      <provideFeedback>1</provideFeedback>
+      <implicitSpringDamper>1</implicitSpringDamper>
+    </gazebo>
     <xacro:shadowarm_lowerarm_transmission />
   </xacro:macro>

File: sr_description/arm/xacro/trunk/shadowarm_trunk.urdf.xacro (robot description, xacro)
@@ -6,5 +6,5 @@
 	  <origin xyz="0 0 0.26525" rpy="0 0 0" />
 	  <mass value="10" />
-	  <inertia  ixx="0.15" ixy="0.0"  ixz="0.0"  iyy="0.15"  iyz="0.0"  izz="0.02" />
+	  <inertia  ixx="0.298" ixy="0.0"  ixz="0.0"  iyy="0.298"  iyz="0.0"  izz="0.0361" />
 	</inertial>
 	<visual>
@@ -35,4 +35,8 @@
       <dynamics damping="5.5"/>
     </joint>
+    <gazebo reference="ShoulderJRotate">
+      <provideFeedback>1</provideFeedback>
+      <implicitSpringDamper>1</implicitSpringDamper>
+    </gazebo>
     <xacro:shadowarm_trunk_transmission />
   </xacro:macro>

File: sr_description/arm/xacro/upper_arm/shadowarm_upperarm.urdf.xacro (robot description, xacro)
@@ -6,5 +6,5 @@
 	<origin xyz="0 0 0.1845" rpy="0 0 0" />
 	<mass value="2" />
-	<inertia  ixx="0.4" ixy="0.0"  ixz="0.0"  iyy="0.4"  iyz="0.0"  izz="0.05" />
+	<inertia  ixx="0.044" ixy="0.0"  ixz="0.0"  iyy="0.044"  iyz="0.0"  izz="0.0056" />
       </inertial>
       <visual>
@@ -34,4 +34,8 @@
       <dynamics damping="5.3"/>
     </joint>
+    <gazebo reference="ShoulderJSwing">
+      <provideFeedback>1</provideFeedback>
+      <implicitSpringDamper>1</implicitSpringDamper>
+    </gazebo>
     <xacro:shadowarm_upperarm_transmission />
   </xacro:macro>

File: sr_description/hand/xacro/finger/biotac/biotac.urdf.xacro (robot description, xacro)
@@ -16,7 +16,7 @@
       <inertial>
         <origin xyz="0 0 0.0125" rpy="0 0 0" />
-        <mass value="0.012" />
-           <inertia  ixx="0.002" ixy="0.0"  ixz="0.0"  iyy="0.002"  iyz="0.0"
-          izz="0.0002" />
+          <mass value="0.017" />
+        <inertia  ixx="0.0000026" ixy="0.0"  ixz="0.0"  iyy="0.0000027"  iyz="0.0"
+        izz="0.00000087" />
       </inertial>
       <visual>
@@ -56,7 +56,11 @@
       <axis xyz="1 0 0" />
       <limit lower="0" upper="${M_PI/2}" effort="2.0"
-      velocity="1.0" />
-      <dynamics damping="0.001"/>
+      velocity="2.0" />
+      <dynamics damping="0.1"/>
     </joint>
+    <gazebo reference="${prefix}${joint_prefix}J2">
+      <provideFeedback>1</provideFeedback>
+      <implicitSpringDamper>1</implicitSpringDamper>
+    </gazebo>
     <link name="${prefix}${link_prefix}_J1_dummy">
       <inertial>
@@ -72,7 +76,11 @@
       <origin xyz="0 0 0.02" rpy="0 0 0" />
       <axis xyz="1 0 0" />
-      <limit lower="${20*M_PI/180}" upper="${20.1*M_PI/180}" effort="1.0" velocity="1.0" />
-      <dynamics damping="0.001"/>
+      <limit lower="${20*M_PI/180}" upper="${20.1*M_PI/180}" effort="1.0" velocity="2.0" />
+      <dynamics damping="0.1"/>
     </joint>
+    <gazebo reference="${prefix}${joint_prefix}J1">
+      <provideFeedback>1</provideFeedback>
+      <implicitSpringDamper>1</implicitSpringDamper>
+    </gazebo>
     <xacro:middle_transmission muscletrans="${muscle}" prefix="${prefix}" joint_prefix="${joint_prefix}" link_prefix="${link_prefix}"/>
     <link name="${prefix}${link_prefix}biotac">
@@ -80,6 +88,6 @@
         <origin xyz="0 0 0" rpy="0 0 0" />
         <mass value="0.040" />
-        <inertia  ixx="0.001" ixy="0.0"  ixz="0.0"  iyy="0.001"  iyz="0.0"
-        izz="0.00025" />
+        <inertia  ixx="0.00000094" ixy="0.0"  ixz="0.0"  iyy="0.0000011"  iyz="0.0"
+        izz="0.00000053" />
       </inertial>
       <visual>

File: sr_description/hand/xacro/finger/distal/distal.gazebo.xacro (robot description, xacro)
@@ -1,5 +1,5 @@
 <?xml version="1.0"?>
 <robot xmlns:xacro="http://ros.org/wiki/xacro">
-  <xacro:macro name="distal_gazebo" params="prefix">
+  <xacro:macro name="distal_gazebo" params="prefix link_prefix">
   <!-- prefix can be anything but usually is "r_" or  "l_" for right and left hands distinction -->
   <gazebo reference="${prefix}${link_prefix}distal">

File: sr_description/hand/xacro/finger/distal/distal.urdf.xacro (robot description, xacro)
@@ -19,7 +19,7 @@
     <link name="${prefix}${link_prefix}distal">
       <inertial>
-        <mass value="0.010" />
+        <mass value="0.012" />
         <origin xyz="0 0 0.012" />
-        <inertia  ixx="0.0000031" ixy="0.0"  ixz="0.0"  iyy="0.0000031"  iyz="0.0"
+        <inertia  ixx="0.00000094" ixy="0.0"  ixz="0.0"  iyy="0.0000011"  iyz="0.0"
         izz="0.00000053" />
       </inertial>
@@ -85,13 +85,17 @@
 				<!-- biotac fixed distal joint -->
         <limit lower="${20/180*M_PI}" upper="${20/180*M_PI}" effort="10"
-          velocity="1.0" />
+          velocity="2.0" />
       </xacro:if>
       <xacro:unless value="${bio}">
 				<!-- standard distal joint -->
         <limit lower="0" upper="${M_PI/2}" effort="2"
-          velocity="1.0" />
+          velocity="2.0" />
       </xacro:unless>
-      <dynamics damping="0.001"/>
+      <dynamics damping="0.1"/>
     </joint>
+    <gazebo reference="${prefix}${joint_prefix}J1">
+      <provideFeedback>1</provideFeedback>
+      <implicitSpringDamper>1</implicitSpringDamper>
+    </gazebo>
     <link name="${prefix}${link_prefix}tip">
 			<inertial>
@@ -108,5 +112,5 @@
     <!-- extensions -->
     <!--   <xacro:distal_transmission muscletrans="${muscle}" prefix="${prefix}" /> -->
-    <xacro:distal_gazebo prefix="${prefix}" />
+    <xacro:distal_gazebo prefix="${prefix}" link_prefix="${link_prefix}"/>
   </xacro:macro>
 </robot>

File: sr_description/hand/xacro/finger/knuckle/knuckle.gazebo.xacro (robot description, xacro)
@@ -1,5 +1,5 @@
 <?xml version="1.0"?>
 <robot xmlns:xacro="http://ros.org/wiki/xacro">
-  <xacro:macro name="knuckle_gazebo" params="prefix">
+  <xacro:macro name="knuckle_gazebo" params="prefix link_prefix">
   <!-- prefix can be anything but usually is "r_" or  "l_" for right and left hands distinction -->
   <gazebo reference="${prefix}${link_prefix}knuckle">

File: sr_description/hand/xacro/finger/knuckle/knuckle.urdf.xacro (robot description, xacro)
@@ -18,6 +18,6 @@
         <origin xyz="0 0 0" rpy="0 0 0" />
         <!--<insert_block name="origin" /> -->
-        <mass value="0.08" />
-        <inertia  ixx="0.000026" ixy="0.0"  ixz="0.0"  iyy="0.000026"  iyz="0.0"	izz="0.000032" />
+        <mass value="0.008" />
+        <inertia  ixx="0.00000026" ixy="0.0"  ixz="0.0"  iyy="0.00000026"  iyz="0.0"	izz="0.00000032" />
       </inertial>
       <visual>
@@ -42,10 +42,14 @@
       <insert_block name="axis"/>
       <limit lower="${-20/180*M_PI}" upper="${20/180*M_PI}"
-      effort="2" velocity="1.0"/>
-      <dynamics damping="0.01"/>
+      effort="2" velocity="2.0"/>
+      <dynamics damping="0.1"/>
     </joint>
+    <gazebo reference="${prefix}${joint_prefix}J4">
+      <provideFeedback>1</provideFeedback>
+      <implicitSpringDamper>1</implicitSpringDamper>
+    </gazebo>
     <!-- extensions -->
     <xacro:knuckle_transmission muscletrans="${muscle}" prefix="${prefix}" joint_prefix="${joint_prefix}" link_prefix="${link_prefix}"/>
-    <xacro:knuckle_gazebo prefix="${prefix}" />
+    <xacro:knuckle_gazebo prefix="${prefix}" link_prefix="${link_prefix}"/>
   </xacro:macro>
 </robot>

File: sr_description/hand/xacro/finger/lfmetacarpal/lfmetacarpal.gazebo.xacro (robot description, xacro)
@@ -1,5 +1,5 @@
 <?xml version="1.0"?>
 <robot xmlns:xacro="http://ros.org/wiki/xacro">
-  <xacro:macro name="lfmetacarpal_gazebo" params="prefix">
+  <xacro:macro name="lfmetacarpal_gazebo" params="prefix link_prefix">
   <!-- prefix can be anything but usually is "r_" or  "l_" for right and left hands distinction -->
   <gazebo reference="${prefix}lfmetacarpal">

File: sr_description/hand/xacro/finger/lfmetacarpal/lfmetacarpal.urdf.xacro (robot description, xacro)
@@ -17,5 +17,5 @@
         <origin xyz="0 0 0.04" rpy="0 0 0" />
         <mass value="0.030" />
-	    <inertia  ixx="0.0000545" ixy="0.0"  ixz="0.0"  iyy="0.000056352"  iyz="0.0" izz="0.000004272" />
+	    <inertia  ixx="0.0000145" ixy="0.0"  ixz="0.0"  iyy="0.00001638"  iyz="0.0" izz="0.000004272" />
       </inertial>
       <visual>
@@ -40,10 +40,14 @@
       <axis xyz="0.573576436 0 ${reflect*0.819152044}" />
         <limit lower="0" upper="${45/180*M_PI}" effort="2"
-      velocity="1.0" />
-      <dynamics damping="0.001"/>
+      velocity="2.0" />
+      <dynamics damping="0.1"/>
     </joint>
+    <gazebo reference="${prefix}LFJ5">
+      <provideFeedback>1</provideFeedback>
+      <implicitSpringDamper>1</implicitSpringDamper>
+    </gazebo>
     <!-- extensions -->
     <xacro:lfmetacarpal_transmission muscletrans="${muscle}" prefix="${prefix}" />
-    <xacro:lfmetacarpal_gazebo prefix="${prefix}" />
+    <xacro:lfmetacarpal_gazebo prefix="${prefix}" link_prefix="${link_prefix}" />
   </xacro:macro>
 </robot>

File: sr_description/hand/xacro/finger/middle/middle.gazebo.xacro (robot description, xacro)
@@ -1,5 +1,5 @@
 <?xml version="1.0"?>
 <robot xmlns:xacro="http://ros.org/wiki/xacro">
-  <xacro:macro name="middle_gazebo" params="prefix">
+  <xacro:macro name="middle_gazebo" params="prefix link_prefix">
   <!-- prefix can be anything but usually is "r_" or  "l_" for right and left hands distinction -->
   <gazebo reference="${prefix}${link_prefix}middle">

File: sr_description/hand/xacro/finger/middle/middle.urdf.xacro (robot description, xacro)
@@ -17,7 +17,7 @@
       <inertial>
         <origin xyz="0 0 0.0125" rpy="0 0 0" />
-        <mass value="0.020" />
-        <inertia  ixx="0.0000067" ixy="0.0"  ixz="0.0"  iyy="0.0000067"  iyz="0.0"
-        izz="0.00000006" />
+        <mass value="0.017" />
+        <inertia  ixx="0.0000026" ixy="0.0"  ixz="0.0"  iyy="0.0000027"  iyz="0.0"
+        izz="0.00000087" />
       </inertial>
       <visual>
@@ -53,10 +53,14 @@
       <axis xyz="1 0 0" />
       <limit lower="0" upper="${M_PI/2}" effort="2"
-      velocity="1.0" />
-      <dynamics damping="0.001"/>
+      velocity="2.0" />
+      <dynamics damping="0.1"/>
     </joint>
+   <gazebo reference="${prefix}${joint_prefix}J2">
+      <provideFeedback>1</provideFeedback>
+      <implicitSpringDamper>1</implicitSpringDamper>
+    </gazebo>
     <!-- extensions -->
     <xacro:middle_transmission muscletrans="${muscle}" prefix="${prefix}" joint_prefix="${joint_prefix}" link_prefix="${link_prefix}"/>
-    <xacro:middle_gazebo prefix="${prefix}" />
+    <xacro:middle_gazebo prefix="${prefix}" link_prefix="${link_prefix}" />
   </xacro:macro>
 </robot>

File: sr_description/hand/xacro/finger/proximal/proximal.gazebo.xacro (robot description, xacro)
@@ -1,5 +1,5 @@
 <?xml version="1.0"?>
 <robot xmlns:xacro="http://ros.org/wiki/xacro">
-  <xacro:macro name="proximal_gazebo" params="prefix">
+  <xacro:macro name="proximal_gazebo" params="prefix link_prefix">
   <!-- prefix can be anything but usually is "r_" or  "l_" for right and left hands distinction -->
   <gazebo reference="${prefix}${link_prefix}proximal">

File: sr_description/hand/xacro/finger/proximal/proximal.urdf.xacro (robot description, xacro)
@@ -18,6 +18,6 @@
         <mass value="0.030" />
         <origin xyz="0 0 0.0225" />
-        <inertia  ixx="0.000037" ixy="0.0"  ixz="0.0"  iyy="0.000037"  iyz="0.0"
-        izz="0.00000018" />
+        <inertia  ixx="0.0000098" ixy="0.0"  ixz="0.0"  iyy="0.00001"  iyz="0.0"
+        izz="0.0000018" />
       </inertial>
       <visual>
@@ -41,10 +41,14 @@
       <axis xyz="1 0 0" />
       <limit lower="0" upper="${M_PI/2}" effort="2"
-      velocity="1.0"/>
-      <dynamics damping="0.001"/>
+      velocity="2.0"/>
+      <dynamics damping="0.1"/>
     </joint>
+    <gazebo reference="${prefix}${joint_prefix}J3">
+      <provideFeedback>1</provideFeedback>
+      <implicitSpringDamper>1</implicitSpringDamper>
+    </gazebo>
     <!-- extensions -->
     <xacro:proximal_transmission muscletrans="${muscle}" prefix="${prefix}" joint_prefix="${joint_prefix}" link_prefix="${link_prefix}"/>
-    <xacro:proximal_gazebo prefix="${prefix}" />
+    <xacro:proximal_gazebo prefix="${prefix}" link_prefix="${link_prefix}"/>
   </xacro:macro>
 </robot>

File: sr_description/hand/xacro/palm/palm.urdf.xacro (robot description, xacro)
@@ -17,5 +17,5 @@
         <origin xyz="0 0 0.035" rpy="0 0 0" />
         <mass value="0.3" />
-        <inertia  ixx="0.0003581" ixy="0.0"  ixz="0.0"  iyy="0.0005287"  iyz="0.0"	izz="0.0002545" />
+        <inertia  ixx="0.0003581" ixy="0.0"  ixz="0.0"  iyy="0.0005287"  iyz="0.0"	izz="0.000191" />
       </inertial>
       <visual>
@@ -81,7 +81,11 @@
       <axis xyz="1 0 0" />
       <limit lower="${-40/180*M_PI}" upper="${28/180*M_PI}"
-      effort="30" velocity="1.0"/>
-      <dynamics damping="0.01"/>
+      effort="30" velocity="2.0"/>
+      <dynamics damping="0.1"/>
     </joint>
+    <gazebo reference="${prefix}WRJ1">
+      <provideFeedback>1</provideFeedback>
+      <implicitSpringDamper>1</implicitSpringDamper>
+    </gazebo>
     <!-- extensions -->
     <xacro:shadowhand_palm_transmission muscletrans="${muscletrans}" prefix="${prefix}" />

File: sr_description/hand/xacro/thumb/thbase.urdf.xacro (robot description, xacro)
@@ -17,5 +17,5 @@
 				<mass value="0.010" />
 				<origin xyz="0 0 0" rpy="0 0 0"/>
-				<inertia  ixx="0.0003" ixy="0.0"  ixz="0.0"  iyy="0.0003"  iyz="0.0" izz="0.0003" />
+				<inertia  ixx="0.00000016" ixy="0.0"  ixz="0.0"  iyy="0.00000016"  iyz="0.0" izz="0.00000016" />
 			</inertial>
       <visual>
@@ -40,8 +40,12 @@
       <origin xyz="${reflect*0.034} -0.0085 0.029" rpy="0 ${M_PI/4} ${M_PI/2-reflect*M_PI/2}" />
       <axis xyz="0 0 ${reflect*-1}" />
-      <limit lower="${-60/180*M_PI}" upper="${60/180*M_PI}" effort="10"
-      velocity="1.0" />
-      <dynamics damping="0.001"/>
+      <limit lower="${-60/180*M_PI}" upper="${60/180*M_PI}" effort="5.0"
+      velocity="4.0" />
+      <dynamics damping="0.2"/>
     </joint>
+    <gazebo reference="${prefix}THJ5">
+      <provideFeedback>1</provideFeedback>
+      <implicitSpringDamper>1</implicitSpringDamper>
+    </gazebo>
     <!-- extensions -->
     <xacro:thbase_transmission muscletrans="${muscle}" prefix="${prefix}"/>

File: sr_description/hand/xacro/thumb/thdistal.urdf.xacro (robot description, xacro)
@@ -20,7 +20,7 @@
 				<inertial>
 					<origin xyz="0 0 0" rpy="0 0 0" />
-					<mass value="0.01" />
-					 <inertia  ixx="0.0007" ixy="0.0"  ixz="0.0"  iyy="0.0007"  iyz="0.0"
-        izz="0.00010" />
+					<mass value="0.008" />
+					 <inertia  ixx="0.0000011" ixy="0.0"  ixz="0.0"  iyy="0.0000011"  iyz="0.0"
+        izz="0.0000005" />
         </inertial>
 			</link>
@@ -30,13 +30,17 @@
 				<origin xyz="0 0 0.02" rpy="0 0 0" />
 				<axis xyz="1 0 0" />
-				<limit lower="${20*M_PI/180}" upper="${20.1*M_PI/180}" effort="10" velocity="0.1" />
-				<dynamics damping="0.001"/>
+				<limit lower="${20*M_PI/180}" upper="${20.1*M_PI/180}" effort="1.0" velocity="4.0" />
+				<dynamics damping="0.2"/>
 			</joint>
+			<gazebo reference="${prefix}THJ1">
+				<provideFeedback>1</provideFeedback>
+				<implicitSpringDamper>1</implicitSpringDamper>
+			</gazebo>
 			<link name="${prefix}thbiotac">
 				<inertial>
 					<origin xyz="0 0 0" rpy="0 0 0" />
-					<mass value="0.2" />
-					 <inertia  ixx="0.0007" ixy="0.0"  ixz="0.0"  iyy="0.0007"  iyz="0.0"
-        izz="0.00010" />
+					<mass value="0.008" />
+					 <inertia  ixx="0.0000011" ixy="0.0"  ixz="0.0"  iyy="0.0000011"  iyz="0.0"
+        izz="0.0000005" />
 				</inertial>
 				<visual>
@@ -113,6 +117,6 @@
 					<mass value="0.016" />
 					<origin xyz="0 0 0.01375" rpy="0 0 0"/>
-					 <inertia  ixx="0.0007" ixy="0.0"  ixz="0.0"  iyy="0.0007"  iyz="0.0"
-        izz="0.00010" />
+					 <inertia  ixx="0.0000021" ixy="0.0"  ixz="0.0"  iyy="0.0000022"  iyz="0.0"
+        izz="0.000001" />
 				</inertial>
 				<visual>
@@ -164,7 +168,11 @@
 				<origin xyz="0 0 0.032" rpy="0 0 ${-M_PI/2}" />
 				<axis xyz="1 0 0" />
-				<limit lower="0" upper="${90.0*M_PI/180}" effort="10" velocity="1.0" />
-				<dynamics damping="0.001"/>
+				<limit lower="0" upper="${90.0*M_PI/180}" effort="1.0" velocity="4.0" />
+				<dynamics damping="0.2"/>
 			</joint>
+			<gazebo reference="${prefix}THJ1">
+				<provideFeedback>1</provideFeedback>
+				<implicitSpringDamper>1</implicitSpringDamper>
+			</gazebo>
 			<link name="${prefix}thtip">
 				<inertial>
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