Commit message: added missing xacro: prefixes

File: sr_description/arm/xacro/base/shadowarm_base.urdf.xacro (robot description, xacro)
@@ -1,4 +1,4 @@
 <robot xmlns:xacro="http://www.ros.org/wiki/xacro">
-<property name="M_PI" value="3.1415926535897931" />
+<xacro:property name="M_PI" value="3.1415926535897931" />
 <xacro:macro name="shadowarm_base">
   <link name="shadowarm_base">

File: sr_description/hand/xacro/ff_biotac_hand.urdf.xacro (robot description, xacro)
@@ -8,5 +8,5 @@
   <xacro:include filename="$(find sr_description)/hand/xacro/finger/fingers.urdf.xacro" />
   <xacro:include filename="$(find sr_description)/hand/xacro/thumb/thumb.urdf.xacro" />
-  <property name="M_PI" value="3.1415926535897931" />
+  <xacro:property name="M_PI" value="3.1415926535897931" />
   <!-- muscletrans is true for muscle transmission to be used, false to use motor transmission -->
   <!-- muscle is true for muscle hand or false for motor hand -->

File: sr_description/hand/xacro/finger/fingers.urdf.xacro (robot description, xacro)
@@ -22,5 +22,5 @@
       <!-- Knuckle -->
       <xacro:knuckle muscle="${muscletrans}" prefix="${prefix}" link_prefix="${link_prefix}" joint_prefix="${joint_prefix}" parent="${prefix}lfmetacarpal" >
-        <insert_block name="origin" />
+        <xacro:insert_block name="origin" />
       </xacro:knuckle>
     </xacro:if>
@@ -29,5 +29,5 @@
       <!-- Knuckle -->
       <xacro:knuckle muscle="${muscletrans}" prefix="${prefix}" link_prefix="${link_prefix}" joint_prefix="${joint_prefix}" parent="${parent}" >
-        <insert_block name="origin" />
+        <xacro:insert_block name="origin" />
       </xacro:knuckle>
     </xacro:unless>

File: sr_description/hand/xacro/finger/knuckle/knuckle.urdf.xacro (robot description, xacro)
@@ -17,5 +17,5 @@
       <inertial>
         <origin xyz="0 0 0" rpy="0 0 0" />
-        <!--<insert_block name="origin" /> -->
+        <!--<xacro:insert_block name="origin" /> -->
         <mass value="0.008" />
         <inertia  ixx="0.00000026" ixy="0.0"  ixz="0.0"  iyy="0.00000026"  iyz="0.0"	izz="0.00000032" />
@@ -39,6 +39,6 @@
       <child link="${prefix}${link_prefix}knuckle"/>
       <!--<origin xyz="0.033 0 0.095" rpy="0 0 0" />-->
-      <insert_block name="origin" />
-      <insert_block name="axis"/>
+      <xacro:insert_block name="origin" />
+      <xacro:insert_block name="axis"/>
       <limit lower="${-20/180*M_PI}" upper="${20/180*M_PI}"
       effort="2" velocity="2.0"/>

File: sr_description/hand/xacro/forearm/forearm_lite.urdf.xacro (robot description, xacro)
@@ -3,5 +3,5 @@
   <!-- prefix can be anything but usually is "r_" or  "l_" for right and left hands distinction -->
   <xacro:macro name="forearm" params="muscle prefix">
-      <property name="M_PI" value="3.1415926535897931" />
+      <xacro:property name="M_PI" value="3.1415926535897931" />
       <link name="${prefix}forearm">
         <inertial>

File: sr_description/hand/xacro/full_hand.tactile.xacro (robot description, xacro)
@@ -5,5 +5,5 @@
   <xacro:include filename="$(find sr_description)/hand/xacro/palm/palm.tactile.xacro" />
   <xacro:include filename="$(find sr_description)/hand/xacro/finger/fingers.tactile.xacro" />
-  <property name="M_PI" value="3.1415926535897931" />
+  <xacro:property name="M_PI" value="3.1415926535897931" />
   <!-- bio is true for biotac finger or false for standard finger -->
   <!-- ubi is true for ubi finger or false for standard finger -->

File: sr_description/hand/xacro/full_hand.urdf.xacro (robot description, xacro)
@@ -8,5 +8,5 @@
   <xacro:include filename="$(find sr_description)/hand/xacro/finger/fingers.urdf.xacro" />
   <xacro:include filename="$(find sr_description)/hand/xacro/thumb/thumb.urdf.xacro" />
-  <property name="M_PI" value="3.1415926535897931" />
+  <xacro:property name="M_PI" value="3.1415926535897931" />
   <!-- muscletrans is true for muscle transmission to be used, false to use motor transmission -->
   <!-- muscle is true for muscle hand or false for motor hand -->

File: sr_description/hand/xacro/hand_lite.urdf.xacro (robot description, xacro)
@@ -8,5 +8,5 @@
   <xacro:include filename="$(find sr_description)/hand/xacro/finger/fingers.urdf.xacro" />
   <xacro:include filename="$(find sr_description)/hand/xacro/thumb/thumb.urdf.xacro" />
-  <property name="M_PI" value="3.1415926535897931" />
+  <xacro:property name="M_PI" value="3.1415926535897931" />
   <!-- muscletrans is true for muscle transmission to be used, false to use motor transmission -->
   <!-- muscle is true for muscle hand or false for motor hand -->

File: sr_description/hand/xacro/one_finger_unit.urdf.xacro (robot description, xacro)
@@ -5,5 +5,5 @@
   <xacro:include filename="$(find sr_description)/hand/xacro/forearm/forearm.urdf.xacro" />
   <xacro:include filename="$(find sr_description)/hand/xacro/finger/fingers.urdf.xacro" />
-  <property name="M_PI" value="3.1415926535897931" />
+  <xacro:property name="M_PI" value="3.1415926535897931" />
   <!-- muscletrans is true for muscle transmission to be used, false to use motor transmission -->
   <!-- muscle is true for muscle hand or false for motor hand -->

File: sr_description/hand/xacro/th_ff_rf_ellipsoid_hand.urdf.xacro (robot description, xacro)
@@ -8,5 +8,5 @@
   <xacro:include filename="$(find sr_description)/hand/xacro/finger/fingers.urdf.xacro" />
   <xacro:include filename="$(find sr_description)/hand/xacro/thumb/thumb.urdf.xacro" />
-  <property name="M_PI" value="3.1415926535897931" />
+  <xacro:property name="M_PI" value="3.1415926535897931" />
   <!-- muscletrans is true for muscle transmission to be used, false to use motor transmission -->
   <!-- muscle is true for muscle hand or false for motor hand -->

File: sr_description/hand/xacro/three_biotac_fingers_hand.urdf.xacro (robot description, xacro)
@@ -8,5 +8,5 @@
   <xacro:include filename="$(find sr_description)/hand/xacro/finger/fingers.urdf.xacro" />
   <xacro:include filename="$(find sr_description)/hand/xacro/thumb/thumb.urdf.xacro" />
-  <property name="M_PI" value="3.1415926535897931" />
+  <xacro:property name="M_PI" value="3.1415926535897931" />
   <!-- muscletrans is true for muscle transmission to be used, false to use motor transmission -->
   <!-- muscle is true for muscle hand or false for motor hand -->

File: sr_description/hand/xacro/three_fingers_hand.urdf.xacro (robot description, xacro)
@@ -8,5 +8,5 @@
   <xacro:include filename="$(find sr_description)/hand/xacro/finger/fingers.urdf.xacro" />
   <xacro:include filename="$(find sr_description)/hand/xacro/thumb/thumb.urdf.xacro" />
-  <property name="M_PI" value="3.1415926535897931" />
+  <xacro:property name="M_PI" value="3.1415926535897931" />
   <!-- muscletrans is true for muscle transmission to be used, false to use motor transmission -->
   <!-- muscle is true for muscle hand or false for motor hand -->

File: sr_description/hand/xacro/wrist/wrist.urdf.xacro (robot description, xacro)
@@ -58,5 +58,5 @@
       <parent link="${parent}"/>
       <child link="${prefix}wrist"/>
-      <insert_block name="origin" />
+      <xacro:insert_block name="origin" />
       <axis xyz="0 ${reflect} 0" />
       <limit lower="${-30/180*M_PI}" upper="${10/180*M_PI}" effort="10" velocity="2.0"/>

File: sr_description/other/xacro/kinect/shadowarm_kinect.urdf.xacro (robot description, xacro)
@@ -1,4 +1,4 @@
 <robot xmlns:xacro="http://ros.org/wiki/xacro">
-  <property name="M_PI" value="3.1415926535"/>
+  <xacro:property name="M_PI" value="3.1415926535"/>
   <xacro:include filename="$(find sr_description)/other/xacro/kinect/gazebo_kinect.urdf.xacro"/>
   <xacro:macro name="shadowarm_side_kinect" params="parent">
