Commit message: Fixed self collision between palm and forearm

File: sr_description/hand/xacro/palm/palm.urdf.xacro (robot description, xacro)
@@ -1,9 +1,9 @@
 <robot xmlns:xacro="http://www.ros.org/wiki/xacro"
-       xmlns:sensor="http://playerstage.sourceforge.net/gazebo/xmlschema/#sensor"
-       xmlns:controller="http://playerstage.sourceforge.net/gazebo/xmlschema/#controller"
-       xmlns:joint="http://playerstage.sourceforge.net/gazebo/xmlschema/#slider"
-       xmlns:interface="http://playerstage.sourceforge.net/gazebo/xmlschema/#interface"
-       xmlns:body="http://playerstage.sourceforge.net/gazebo/xmlschema/#body"
-       xmlns:geom="http://playerstage.sourceforge.net/gazebo/xmlschema/#geom">
+xmlns:sensor="http://playerstage.sourceforge.net/gazebo/xmlschema/#sensor"
+xmlns:controller="http://playerstage.sourceforge.net/gazebo/xmlschema/#controller"
+xmlns:joint="http://playerstage.sourceforge.net/gazebo/xmlschema/#slider"
+xmlns:interface="http://playerstage.sourceforge.net/gazebo/xmlschema/#interface"
+xmlns:body="http://playerstage.sourceforge.net/gazebo/xmlschema/#body"
+xmlns:geom="http://playerstage.sourceforge.net/gazebo/xmlschema/#geom">
   <xacro:include filename="$(find sr_description)/hand/xacro/palm/palm.gazebo.xacro" />
   <xacro:include filename="$(find sr_description)/hand/xacro/palm/palm.transmission.xacro" />
@@ -12,10 +12,12 @@
   <!-- reflect is either 1 (for right hand) or -1 (for left hand) -->
   <!-- parent is the parent link for the joint -->
-  <xacro:macro name="palm" params="muscletrans prefix reflect parent">
+  <xacro:macro name="palm"
+  params="muscletrans prefix reflect parent">
     <link name="${prefix}palm">
       <inertial>
         <origin xyz="0 0 0.035" rpy="0 0 0" />
         <mass value="0.3" />
-        <inertia  ixx="0.0003581" ixy="0.0"  ixz="0.0"  iyy="0.0005287"  iyz="0.0"	izz="0.000191" />
+        <inertia ixx="0.0003581" ixy="0.0" ixz="0.0"
+        iyy="0.0005287" iyz="0.0" izz="0.000191" />
       </inertial>
       <visual>
@@ -23,7 +25,7 @@
         <geometry name="${prefix}palm_visual">
           <mesh filename="package://sr_description/hand/model/palm.dae"
-					 scale="${reflect*0.001} 0.001 0.001" />
+          scale="${reflect*0.001} 0.001 0.001" />
         </geometry>
-        <material name="Grey"/>
+        <material name="Grey" />
       </visual>
       <collision>
@@ -34,19 +36,29 @@
       </collision>
       <collision>
-        <origin xyz="${reflect*0.0005} -0.0035 0.038" rpy="0 0 0" />
+        <origin xyz="${-reflect*0.002} -0.0035 0.038"
+        rpy="0 0 0" />
         <geometry>
-          <box size="0.041 0.017 0.098" />
+          <box size="0.036 0.017 0.098" />
         </geometry>
       </collision>
       <!-- palm complement below first finger -->
       <collision>
-        <origin xyz="${reflect*0.0315} -0.0035 0.073" rpy="0 0 0" />
+        <origin xyz="${reflect*0.029} -0.0035 0.082"
+        rpy="0 0 0" />
         <geometry>
-          <box size="0.021 0.017 0.028" />
+          <box size="0.026 0.017 0.010" />
+        </geometry>
+      </collision>
+      <collision>
+        <origin xyz="${reflect*0.0265} -0.001 0.070"
+        rpy="0.2 0 ${reflect*0.25}" />
+        <geometry>
+          <box size="0.026 0.014 0.018" />
         </geometry>
       </collision>
       <!-- thumb pulp side -->
       <collision>
-        <origin xyz="${reflect*0.0315} -0.0085 0.001" rpy="0 0 0" />
+        <origin xyz="${reflect*0.0315} -0.0085 0.001"
+        rpy="0 0 0" />
         <geometry>
           <box size="0.021 0.027 0.024" />
@@ -55,7 +67,7 @@
       <!-- thumb pulp central -->
       <collision>
-        <origin xyz="${reflect*0.01} -0.017 0.011" rpy="0 0 0" />
+        <origin xyz="${reflect*0.0125} -0.015 0.009" rpy="0 0 ${reflect*-0.48}" />
         <geometry>
-          <box size="0.022 0.010 0.044" />
+          <box size="0.022 0.005 0.040" />
         </geometry>
       </collision>
@@ -70,17 +82,17 @@
       <collision>
         <origin xyz="${reflect*-0.030} 0 0.009" rpy="0 0 0" />
-	      <geometry>
-            <box size="0.020 0.024 0.040" />
-          </geometry>
+        <geometry>
+          <box size="0.020 0.024 0.040" />
+        </geometry>
       </collision>
     </link>
     <joint name="${prefix}WRJ1" type="revolute">
-      <parent link="${parent}"/>
-      <child link="${prefix}palm"/>
+      <parent link="${parent}" />
+      <child link="${prefix}palm" />
       <origin xyz="0 0 0.034" rpy="0 0 0" />
       <axis xyz="1 0 0" />
       <limit lower="${-40/180*M_PI}" upper="${28/180*M_PI}"
-      effort="30" velocity="2.0"/>
-      <dynamics damping="0.1"/>
+      effort="30" velocity="2.0" />
+      <dynamics damping="0.1" />
     </joint>
     <gazebo reference="${prefix}WRJ1">
@@ -89,5 +101,6 @@
     </gazebo>
     <!-- extensions -->
-    <xacro:shadowhand_palm_transmission muscletrans="${muscletrans}" prefix="${prefix}" />
+    <xacro:shadowhand_palm_transmission muscletrans="${muscletrans}"
+    prefix="${prefix}" />
     <xacro:shadowhand_palm_gazebo prefix="${prefix}" />
   </xacro:macro>
