Commit message: adapted to new argument forwarding syntax ($|)

File: sr_description/hand/xacro/finger/fingers.tactile.ubi.xacro (robot description, xacro)
@@ -8,8 +8,7 @@
        normals: create tags for arrow markers?
   -->
-  <!-- prefix can be anything but usually is "r_" or  "l_" for right and left hands distinction -->
-  <!-- link_prefix prepends fingername to the link names -->
-  <!-- finger_number is the finger index in the distal tactile message -->
-  <xacro:macro name="finger_tactile" params="prefix finger reflect meshes normals">
+  <xacro:macro name="finger_tactile"
+               params="prefix:=$|'' reflect:=$|1 finger
+                       meshes:=$|1 normals:=$|1">
     <xacro:property name="finger_no" value="${dict(ff=0, mf=1, rf=2, lf=3)}"/>
     <xacro:property name="ns" value="${prefix}${finger}"/>

File: sr_description/hand/xacro/full_hand.tactile.xacro (robot description, xacro)
@@ -2,5 +2,4 @@
   <!-- Create mesh and arrow markers for a single taxel.
        Expected parameters:
-       meshes + normals = 0 | 1
        topic: ROS topic
        data: data field in ROS topic stream
@@ -8,11 +7,15 @@
        ns:   marker namespace in rviz
        xs:   raw sensor range
+       taxel_data: dict of taxel positions and normals
        mesh: mesh resource
        mesh_scale: 3-dim vector for mesh scaling
-       normal_scale
+       arrow_scale: 4-dim scaling vector:
+                    len scaling, shaft thickness, head thickness, head len
+       meshes + normals = 0 | 1
   -->
-  <xacro:macro name="xacro:tactile" params="topic data link ns xs
-                                            mesh mesh_scale arrow_scale
-                                            meshes normals">
+  <xacro:macro name="xacro:tactile"
+               params="topic:=$ data link:=$ ns:=$ xs:=$ taxel_data:=$
+                       mesh:=$ mesh_scale:=$ arrow_scale:=$
+                       meshes:=$ normals:=$">
     <!-- extract channel number -->
     <xacro:property name="channel" value="${data[:-1].rsplit('[',1)[1]}"/>
@@ -45,5 +48,6 @@
        normals: create tags for arrow markers?
   -->
-  <xacro:macro name="shadowhand_tactile" params="tactile reflect:=1 prefix:='' meshes normals">
+  <xacro:macro name="shadowhand_tactile"
+               params="tactile:=$ reflect:=$|1 prefix:=$|'' meshes:=$ normals:=$">
     <xacro:include filename="$(find sr_description)/hand/xacro/palm/palm.tactile.${tactile}.xacro"/>
     <xacro:include filename="$(find sr_description)/hand/xacro/finger/fingers.tactile.${tactile}.xacro"/>

File: sr_description/hand/xacro/palm/palm.tactile.ubi.xacro (robot description, xacro)
@@ -1,5 +1,11 @@
 <robot xmlns:xacro="http://www.ros.org/wiki/xacro">
-  <!-- prefix can be anything but usually is "r_" or  "l_" for right and left hands distinction -->
-  <xacro:macro name="palm_tactile" params="prefix reflect meshes:=1 normals:=0">
+  <!-- Create <tactile> tags for a single finger
+       prefix:  hand prefix, usually rh_ or lh_
+       reflect: +1 / -1 to indicate right / left hand
+       meshes:  create tags for mesh markers?
+       normals: create tags for arrow markers?
+  -->
+  <xacro:macro name="palm_tactile"
+               params="prefix:=$|'' reflect:=$|1 meshes:=$|1 normals:=$|1">
     <!-- link parameters -->
     <xacro:property name="ns" value="${prefix}palm"/>

File: sr_description/hand/xacro/thumb/thumb.tactile.ubi.xacro (robot description, xacro)
@@ -1,5 +1,4 @@
 <robot xmlns:xacro="http://www.ros.org/wiki/xacro">
   <!-- Create <tactile> tags for a single finger
-       tactile: sensor type
        prefix:  hand prefix, usually rh_ or lh_
        reflect: +1 / -1 to indicate right / left hand
@@ -7,8 +6,6 @@
        normals: create tags for arrow markers?
   -->
-  <!-- prefix can be anything but usually is "r_" or  "l_" for right and left hands distinction -->
-  <!-- link_prefix prepends fingername to the link names -->
-  <!-- finger_number is the finger index in the distal tactile message -->
-  <xacro:macro name="thumb_tactile" params="prefix reflect meshes normals">
+  <xacro:macro name="thumb_tactile"
+               params="prefix:=$|'' reflect:=$|1 meshes:=$|1 normals:=$|1">
     <xacro:property name="ns" value="${prefix}th"/>
     <xacro:property name="taxel_dir" value="$(find sr_description)/hand/xacro/thumb/"/>

Commit message: reduced sensor range for fabrics-based tactile sensors

File: sr_description/hand/xacro/finger/fingers.tactile.ubi.xacro (robot description, xacro)
@@ -25,5 +25,5 @@
     <xacro:property name="data" value="sensors[${finger_no[finger]}]/proximal"/>
     <xacro:property name="link" value="${prefix}${finger}proximal"/>
-    <xacro:property name="xs" value="0 4095"/>
+    <xacro:property name="xs" value="0 2047"/>
     <xacro:tactile data="${data}[0]"  mesh="${mesh_dir}/tax_prox_r.stl"/>
     <xacro:tactile data="${data}[1]" mesh="${mesh_dir}/tax_prox_m.stl"/>

File: sr_description/hand/xacro/palm/palm.tactile.ubi.xacro (robot description, xacro)
@@ -11,5 +11,5 @@
     <xacro:property name="ns" value="${prefix}palm"/>
     <!-- tactile data parameters -->
-    <xacro:property name="xs" value="0 4095"/>
+    <xacro:property name="xs" value="0 2047"/>
     <xacro:property name="taxel_dir" value="$(find sr_description)/hand/xacro/palm"/>
     <!-- mesh parameters -->
