Commit message: reworked tactile marker description for UBI taxels
added arrow markers (taxel position+normals from yaml config)
prepared for thumb

File: sr_description/hand/xacro/full_hand.tactile.xacro (robot description, xacro)
@@ -1,24 +1,64 @@
-<robot xmlns:sensor="http://playerstage.sourceforge.net/gazebo/xmlschema/#sensor"
-       xmlns:controller="http://playerstage.sourceforge.net/gazebo/xmlschema/#controller"
-       xmlns:interface="http://playerstage.sourceforge.net/gazebo/xmlschema/#interface"
-       xmlns:xacro="http://www.ros.org/wiki/xacro">
-  <xacro:include filename="$(find sr_description)/hand/xacro/palm/palm.tactile.xacro" />
-  <xacro:include filename="$(find sr_description)/hand/xacro/finger/fingers.tactile.xacro" />
-  <xacro:property name="M_PI" value="3.1415926535897931" />
-  <!-- bio is true for biotac finger or false for standard finger -->
-  <!-- ubi is true for ubi finger or false for standard finger -->
-  <!-- eli is true for ellipsoid fingertip or false for standard finger -->
-  <!-- prefix can be anything but usually is "r_" or  "l_" for right and left hands distinction -->
-  <xacro:macro name="shadowhand_tactile" params="bio ubi eli reflect prefix">
+<robot xmlns:xacro="http://www.ros.org/wiki/xacro">
+  <!-- Create mesh and arrow markers for a single taxel.
+       Expected parameters:
+       meshes + normals = 0 | 1
+       topic: ROS topic
+       data: data field in ROS topic stream
+       link: link name
+       ns:   marker namespace in rviz
+       xs:   raw sensor range
+       mesh: mesh resource
+       mesh_scale: 3-dim vector for mesh scaling
+       normal_scale
+  -->
+  <xacro:macro name="xacro:tactile" params="topic data link ns xs
+                                            mesh mesh_scale arrow_scale
+                                            meshes normals">
+    <!-- extract channel number -->
+    <xacro:property name="channel" value="${data[:-1].rsplit('[',1)[1]}"/>
+    <xacro:if value="${meshes}">
+      <!-- mesh marker -->
+      <tactile topic="${topic}" data="${data}"
+               link="${link}" ns="meshes/${ns}" xs="${xs}">
+        <origin xyz="0 0 0" rpy="0 0 0"/>
+        <geometry>
+          <mesh filename="${mesh}" scale="${mesh_scale}" />
+        </geometry>
+      </tactile>
+    </xacro:if>
+    <xacro:if value="${normals}">
+      <!-- arrow marker -->
+      <tactile topic="${topic}" data="${data}" link="${link}" ns="normals/${ns}" xs="${xs}">
+        <origin xyz="${' '.join([str(v) for v in taxel_data['positions'][channel]])}"/>
+        <geometry>
+          <arrow dir="${' '.join([str(v) for v in taxel_data['normals'][channel]])}"
+                 scale="${arrow_scale}"/>
+        </geometry>
+      </tactile>
+    </xacro:if>
+  </xacro:macro>
+  <!-- Create <tactile> tags describing the taxels
+       tactile: sensor type
+       prefix:  hand prefix, usually rh_ or lh_
+       reflect: +1 / -1 to indicate right / left hand
+       meshes:  create tags for mesh markers?
+       normals: create tags for arrow markers?
+  -->
+  <xacro:macro name="shadowhand_tactile" params="tactile reflect:=1 prefix:='' meshes normals">
+    <xacro:include filename="$(find sr_description)/hand/xacro/palm/palm.tactile.${tactile}.xacro"/>
+    <xacro:include filename="$(find sr_description)/hand/xacro/finger/fingers.tactile.${tactile}.xacro"/>
+    <xacro:include filename="$(find sr_description)/hand/xacro/thumb/thumb.tactile.${tactile}.xacro"/>
     <!-- Palm -->
-    <xacro:palm_tactile reflect="${reflect}" prefix="${prefix}" />
+    <xacro:palm_tactile normals="0"/>
     <!-- First Finger -->
-    <xacro:finger_tactile lf="false" bio="${bio}" ubi="${ubi}" eli="${eli}" reflect="${reflect}" prefix="${prefix}" link_prefix="ff"  finger_number="0"/>
+    <xacro:finger_tactile finger="ff"/>
     <!-- Middle Finger -->
-    <xacro:finger_tactile lf="false" bio="${bio}" ubi="${ubi}" eli="${eli}" reflect="${reflect}" prefix="${prefix}" link_prefix="mf"  finger_number="1"/>
+    <xacro:finger_tactile finger="mf"/>
     <!-- Ring Finger -->
-    <xacro:finger_tactile lf="false" bio="${bio}" ubi="${ubi}" eli="${eli}" reflect="${reflect}" prefix="${prefix}" link_prefix="rf"  finger_number="2"/>
+    <xacro:finger_tactile finger="rf"/>
     <!-- Little Finger  -->
-    <xacro:finger_tactile lf="true" bio="${bio}" ubi="${ubi}" eli="${eli}" reflect="${reflect}" prefix="${prefix}" link_prefix="lf"  finger_number="3"/>
+    <xacro:finger_tactile finger="lf"/>
+    <!-- Thumb  -->
+    <xacro:thumb_tactile/>
   </xacro:macro>
 </robot>

Commit message: Added normals and positions for palm and metacarpal taxels

File: sr_description/hand/xacro/full_hand.tactile.xacro (robot description, xacro)
@@ -50,5 +50,5 @@
     <xacro:include filename="$(find sr_description)/hand/xacro/thumb/thumb.tactile.${tactile}.xacro"/>
     <!-- Palm -->
-    <xacro:palm_tactile normals="0"/>
+    <xacro:palm_tactile />
     <!-- First Finger -->
     <xacro:finger_tactile finger="ff"/>

File: sr_description/hand/xacro/palm/palm.tactile.ubi.xacro (robot description, xacro)
@@ -6,4 +6,5 @@
     <!-- tactile data parameters -->
     <xacro:property name="xs" value="0 4095"/>
+    <xacro:property name="taxel_dir" value="$(find sr_description)/hand/xacro/palm"/>
     <!-- mesh parameters -->
     <xacro:property name="dir" value="package://sr_description/hand/model/ubi_tactiles"/>
@@ -11,4 +12,5 @@
     <!-- arrow parameters -->
     <xacro:property name="arrow_scale" value="0.01 0.0005 0.001"/>
+    <xacro:property name="taxel_data" value="${load_yaml(taxel_dir + '/metacarpal.taxels.ubi.yaml')}"/>
     <xacro:property name="topic" value="palm_extras"/>
     <xacro:property name="link" value="${prefix}lfmetacarpal"/>
@@ -18,4 +20,5 @@
     <xacro:property name="link" value="${prefix}palm"/>
     <xacro:tactile data="data[9]" mesh="${dir}/tax_palm_side.stl"/>
+    <xacro:property name="taxel_data" value="${load_yaml(taxel_dir + '/palm.taxels.ubi.yaml')}"/>
     <xacro:property name="topic" value="tactile_aux_spi"/>
     <xacro:tactile data="sensors[0]" mesh="${dir}/tax_palm_up_r.stl"/>

Commit message: cleanup: removed old xacro:tactile macro (was replaced by xacro:taxel)

File: sr_description/hand/xacro/full_hand.tactile.xacro (robot description, xacro)
@@ -1,44 +1,3 @@
 <robot xmlns:xacro="http://www.ros.org/wiki/xacro">
-  <!-- Create mesh and arrow markers for a single taxel.
-       Expected parameters:
-       topic: ROS topic
-       data: data field in ROS topic stream
-       link: link name
-       ns:   marker namespace in rviz
-       xs:   raw sensor range
-       taxel_data: dict of taxel positions and normals
-       mesh: mesh resource
-       mesh_scale: 3-dim vector for mesh scaling
-       arrow_scale: 4-dim scaling vector:
-                    len scaling, shaft thickness, head thickness, head len
-       meshes + normals = 0 | 1
-  -->
-  <xacro:macro name="xacro:tactile"
-               params="topic:=$ data link:=$ ns:=$ xs:=$ taxel_data:=$
-                       mesh:=$ mesh_scale:=$ arrow_scale:=$
-                       meshes:=$ normals:=$">
-    <!-- extract channel number -->
-    <xacro:property name="channel" value="${data[:-1].rsplit('[',1)[1]}"/>
-    <xacro:if value="${meshes}">
-      <!-- mesh marker -->
-      <tactile topic="${topic}" data="${data}"
-               link="${link}" ns="meshes/${ns}" xs="${xs}">
-        <origin xyz="0 0 0" rpy="0 0 0"/>
-        <geometry>
-          <mesh filename="${mesh}" scale="${mesh_scale}" />
-        </geometry>
-      </tactile>
-    </xacro:if>
-    <xacro:if value="${normals}">
-      <!-- arrow marker -->
-      <tactile topic="${topic}" data="${data}" link="${link}" ns="normals/${ns}" xs="${xs}">
-        <origin xyz="${' '.join([str(v) for v in taxel_data['positions'][channel]])}"/>
-        <geometry>
-          <arrow dir="${' '.join([str(v) for v in taxel_data['normals'][channel]])}"
-                 scale="${arrow_scale}"/>
-        </geometry>
-      </tactile>
-    </xacro:if>
-  </xacro:macro>
   <!-- Create <tactile> tags describing the taxels
        tactile: sensor type

File: sr_description/hand/xacro/tactile.ubi.xacro (robot description, xacro)
@@ -80,5 +80,5 @@
     <!-- Middle -->
     <xacro:middle_tactile taxel_data="${load_yaml(taxel_dir + '/middle/middle.taxels.ubi.yaml')}"/>
-    <!-- Distal  -->
+    <!-- Distal -->
     <xacro:property name="xs" value="1023 0"/>
     <xacro:distal_tactile taxel_data="${load_yaml(taxel_dir + '/distal/distal.taxels.ubi.yaml')}"/>
@@ -104,20 +104,20 @@
     <xacro:property name="mesh_scale" value="${reflect*0.00101} 0.00101 0.00101"/>
     <!-- taxels attached to lfmetacarpal -->
-    <xacro:tactile data="data[6]" mesh="${mesh_dir}/tax_metac_upper.stl"/>
-    <xacro:tactile data="data[7]" mesh="${mesh_dir}/tax_metac_lower.stl"/>
-    <xacro:tactile data="data[8]" mesh="${mesh_dir}/tax_metac_side.stl"/>
+    <xacro:taxel data="data[6]" mesh="${mesh_dir}/tax_metac_upper.stl"/>
+    <xacro:taxel data="data[7]" mesh="${mesh_dir}/tax_metac_lower.stl"/>
+    <xacro:taxel data="data[8]" mesh="${mesh_dir}/tax_metac_side.stl"/>
     <!-- taxels attached to palm -->
     <xacro:property name="link" value="${prefix}palm"/>
-    <xacro:tactile data="data[9]" mesh="${mesh_dir}/tax_palm_side.stl"/>
+    <xacro:taxel data="data[9]" mesh="${mesh_dir}/tax_palm_side.stl"/>
     <xacro:property name="taxel_data" value="${load_yaml(taxel_dir + '/palm.taxels.ubi.yaml')}"/>
     <xacro:property name="topic" value="tactile_aux_spi"/>
-    <xacro:tactile data="sensors[0]" mesh="${mesh_dir}/tax_palm_up_r.stl"/>
-    <xacro:tactile data="sensors[1]" mesh="${mesh_dir}/tax_palm_up_mid.stl"/>
-    <xacro:tactile data="sensors[2]" mesh="${mesh_dir}/tax_palm_up_l.stl"/>
-    <xacro:tactile data="sensors[3]" mesh="${mesh_dir}/tax_palm_center_r.stl"/>
-    <xacro:tactile data="sensors[4]" mesh="${mesh_dir}/tax_palm_center_l.stl"/>
-    <xacro:tactile data="sensors[5]" mesh="${mesh_dir}/tax_palm_center_mid.stl"/>
-    <xacro:tactile data="sensors[6]" mesh="${mesh_dir}/tax_palm_down_r.stl"/>
-    <xacro:tactile data="sensors[7]" mesh="${mesh_dir}/tax_palm_down_l.stl"/>
+    <xacro:taxel data="sensors[0]" mesh="${mesh_dir}/tax_palm_up_r.stl"/>
+    <xacro:taxel data="sensors[1]" mesh="${mesh_dir}/tax_palm_up_mid.stl"/>
+    <xacro:taxel data="sensors[2]" mesh="${mesh_dir}/tax_palm_up_l.stl"/>
+    <xacro:taxel data="sensors[3]" mesh="${mesh_dir}/tax_palm_center_r.stl"/>
+    <xacro:taxel data="sensors[4]" mesh="${mesh_dir}/tax_palm_center_l.stl"/>
+    <xacro:taxel data="sensors[5]" mesh="${mesh_dir}/tax_palm_center_mid.stl"/>
+    <xacro:taxel data="sensors[6]" mesh="${mesh_dir}/tax_palm_down_r.stl"/>
+    <xacro:taxel data="sensors[7]" mesh="${mesh_dir}/tax_palm_down_l.stl"/>
   </xacro:macro>
 </robot>
